File: BoostConverter/InverterBoostConverter/PhaseA.kicad_sch (KiCad schematic)
At the start: 34 parts, among them IC8 LM358DR, Q1 IMBG65R015M2H, Q4 IMBG65R015M2H, U6 ACS758xCB-200U-PFF

Commit message: Finish Boost Converter
Parts:
- C35, C47, C71, C72, C73, C74, C75: footprint 1210 -> Capacitor_SMD:C_1210_3225Metric_Pad1.33x2.70mm_HandSolder
- D1, D10, D18, D19, D2, D5, D6, D7, D8, D9: footprint VS30CDU06HM3I -> InverterCom:VS30CDU06HM3I
- FB1, FB3: footprint BEADC1608X100N -> InverterCom:BEADC1608X100N
- IC8: footprint SOIC127P600X175-8N -> InverterCom:SOIC127P600X175-8N
- L1, L3, L4, L5, L6, L7: footprint IHDM1008BCEV2R2M20 -> InverterCom:IHDM1008BCEV2R2M20
- Q1, Q4: footprint (none) -> InverterCom:TO127P1500X470-8N-2-V1
- R39, R51, R52, R55, R56: footprint 1210 -> Resistor_SMD:R_1210_3225Metric_Pad1.30x2.65mm_HandSolder
Changed lines of the file:
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@@
 			)
 		)
-		(property "Footprint" "IHDM1008BCEV2R2M20"
+		(property "Footprint" "InverterCom:IHDM1008BCEV2R2M20"
 			(at 109.22 174.93 0)
 			(effects
@@
 			)
 		)
-		(property "Footprint" ""
+		(property "Footprint" "InverterCom:TO127P1500X470-8N-2-V1"
 			(at 180.34 111.76 0)
 			(effects
@@
 			)
 		)
-		(property "Footprint" "VS30CDU06HM3I"
+		(property "Footprint" "InverterCom:VS30CDU06HM3I"
 			(at 256.54 90.17 0)
 			(effects
@@
 			)
 		)
-		(property "Footprint" "1210"
+		(property "Footprint" "Resistor_SMD:R_1210_3225Metric_Pad1.30x2.65mm_HandSolder"
 			(at 144.272 119.38 90)
 			(effects
@@
 			)
 		)
-		(property "Footprint" "BEADC1608X100N"
+		(property "Footprint" "InverterCom:BEADC1608X100N"
 			(at 97.79 116.078 90)
 			(effects
@@
 			)
 		)
-		(property "Footprint" "1210"
+		(property "Footprint" "Capacitor_SMD:C_1210_3225Metric_Pad1.33x2.70mm_HandSolder"
 			(at 100.6348 115.57 0)
 			(effects
@@
 			)
 		)
-		(property "Footprint" "1210"
+		(property "Footprint" "Capacitor_SMD:C_1210_3225Metric_Pad1.33x2.70mm_HandSolder"
 			(at 235.9152 33.02 0)
 			(effects
@@
 			)
 		)
-		(property "Footprint" "VS30CDU06HM3I"
+		(property "Footprint" "InverterCom:VS30CDU06HM3I"
 			(at 256.54 76.2 0)
 			(effects
@@
 			)
 		)
-		(property "Footprint" "VS30CDU06HM3I"
+		(property "Footprint" "InverterCom:VS30CDU06HM3I"
 			(at 54.61 48.26 0)
 			(effects
@@
 			)
 		)
-		(property "Footprint" "1210"
+		(property "Footprint" "Resistor_SMD:R_1210_3225Metric_Pad1.30x2.65mm_HandSolder"
 			(at 84.582 119.38 90)
 			(effects
@@
 			)
 		)
-		(property "Footprint" "1210"
+		(property "Footprint" "Capacitor_SMD:C_1210_3225Metric_Pad1.33x2.70mm_HandSolder"
 			(at 158.4452 53.34 0)
 			(effects
@@
 			)
 		)
-		(property "Footprint" "BEADC1608X100N"
+		(property "Footprint" "InverterCom:BEADC1608X100N"
 			(at 157.48 116.078 90)
 			(effects
@@
 			)
 		)
-		(property "Footprint" "1210"
+		(property "Footprint" "Resistor_SMD:R_1210_3225Metric_Pad1.30x2.65mm_HandSolder"
 			(at 84.582 130.81 90)
 			(effects
@@
 			)
 		)
-		(property "Footprint" "VS30CDU06HM3I"
+		(property "Footprint" "InverterCom:VS30CDU06HM3I"
 			(at 54.61 62.23 0)
 			(effects
@@
 			)
 		)
-		(property "Footprint" "IHDM1008BCEV2R2M20"
+		(property "Footprint" "InverterCom:IHDM1008BCEV2R2M20"
 			(at 109.22 185.09 0)
 			(effects
@@
 			)
 		)
-		(property "Footprint" "IHDM1008BCEV2R2M20"
+		(property "Footprint" "InverterCom:IHDM1008BCEV2R2M20"
 			(at 109.22 164.77 0)
 			(effects
@@
 			)
 		)
-		(property "Footprint" "VS30CDU06HM3I"
+		(property "Footprint" "InverterCom:VS30CDU06HM3I"
 			(at 54.61 76.2 0)
 			(effects
@@
 			)
 		)
-		(property "Footprint" ""
+		(property "Footprint" "InverterCom:TO127P1500X470-8N-2-V1"
 			(at 120.65 111.76 0)
 			(effects
@@
 			)
 		)
-		(property "Footprint" "IHDM1008BCEV2R2M20"
+		(property "Footprint" "InverterCom:IHDM1008BCEV2R2M20"
 			(at 86.36 185.09 0)
 			(effects
@@
 			)
 		)
-		(property "Footprint" "1210"
+		(property "Footprint" "Resistor_SMD:R_1210_3225Metric_Pad1.30x2.65mm_HandSolder"
 			(at 144.272 130.81 90)
 			(effects
@@
 			)
 		)
-		(property "Footprint" "VS30CDU06HM3I"
+		(property "Footprint" "InverterCom:VS30CDU06HM3I"
 			(at 256.54 132.08 0)
 			(effects
@@
 			)
 		)
-		(property "Footprint" "1210"
+		(property "Footprint" "Capacitor_SMD:C_1210_3225Metric_Pad1.33x2.70mm_HandSolder"
 			(at 223.2152 33.02 0)
 			(effects
@@
 			)
 		)
-		(property "Footprint" "SOIC127P600X175-8N"
+		(property "Footprint" "InverterCom:SOIC127P600X175-8N"
 			(at 217.17 130.48 0)
 			(effects
@@
 			)
 		)
-		(property "Footprint" "VS30CDU06HM3I"
+		(property "Footprint" "InverterCom:VS30CDU06HM3I"
 			(at 256.54 62.23 0)
 			(effects
@@
 			)
 		)
-		(property "Footprint" "VS30CDU06HM3I"
+		(property "Footprint" "InverterCom:VS30CDU06HM3I"
 			(at 54.61 34.29 0)
 			(effects
@@
 			)
 		)
-		(property "Footprint" "1210"
+		(property "Footprint" "Capacitor_SMD:C_1210_3225Metric_Pad1.33x2.70mm_HandSolder"
 			(at 145.7452 53.34 0)
 			(effects
@@
 			)
 		)
-		(property "Footprint" "VS30CDU06HM3I"
+		(property "Footprint" "InverterCom:VS30CDU06HM3I"
 			(at 256.54 104.14 0)
 			(effects
@@
 			)
 		)
-		(property "Footprint" "1210"
+		(property "Footprint" "Capacitor_SMD:C_1210_3225Metric_Pad1.33x2.70mm_HandSolder"
 			(at 160.3248 115.57 0)
 			(effects
@@
 			)
 		)
-		(property "Footprint" "IHDM1008BCEV2R2M20"
+		(property "Footprint" "InverterCom:IHDM1008BCEV2R2M20"
 			(at 86.36 174.93 0)
 			(effects
@@
 			)
 		)
-		(property "Footprint" "1210"
+		(property "Footprint" "Resistor_SMD:R_1210_3225Metric_Pad1.30x2.65mm_HandSolder"
 			(at 171.45 72.898 90)
 			(effects
@@
 			)
 		)
-		(property "Footprint" "VS30CDU06HM3I"
+		(property "Footprint" "InverterCom:VS30CDU06HM3I"
 			(at 256.54 118.11 0)
 			(effects
@@
 			)
 		)
-		(property "Footprint" "1210"
+		(property "Footprint" "Capacitor_SMD:C_1210_3225Metric_Pad1.33x2.70mm_HandSolder"
 			(at 177.4952 80.01 0)
 			(effects
@@
 			)
 		)
-		(property "Footprint" "IHDM1008BCEV2R2M20"
+		(property "Footprint" "InverterCom:IHDM1008BCEV2R2M20"
 			(at 86.36 164.77 0)
 			(effects
