File: BoostConverter/InverterBoostConverter/PhaseB.kicad_sch (KiCad schematic)
At the start: 34 parts, among them IC9 LM358DR, Q2 IMBG65R015M2H, Q5 IMBG65R015M2H, U1 ACS758xCB-200U-PFF

Commit message: Finish Boost Converter
Parts:
- C36, C48, C76, C77, C78, C79, C80: footprint 1210 -> Capacitor_SMD:C_1210_3225Metric_Pad1.33x2.70mm_HandSolder
- D11, D12, D13, D14, D15, D16, D17, D20, D3, D4: footprint VS30CDU06HM3I -> InverterCom:VS30CDU06HM3I
- FB2, FB4: footprint BEADC1608X100N -> InverterCom:BEADC1608X100N
- IC9: footprint SOIC127P600X175-8N -> InverterCom:SOIC127P600X175-8N
- L10, L11, L12, L2, L8, L9: footprint IHDM1008BCEV2R2M20 -> InverterCom:IHDM1008BCEV2R2M20
- Q2, Q5: footprint (none) -> InverterCom:TO127P1500X470-8N-2-V1
- R40, R45, R46, R53, R54: footprint 1210 -> Resistor_SMD:R_1210_3225Metric_Pad1.30x2.65mm_HandSolder
Changed lines of the file:
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@@
 			)
 		)
-		(property "Footprint" "1210"
+		(property "Footprint" "Capacitor_SMD:C_1210_3225Metric_Pad1.33x2.70mm_HandSolder"
 			(at 95.5548 121.92 0)
 			(effects
@@
 			)
 		)
-		(property "Footprint" "IHDM1008BCEV2R2M20"
+		(property "Footprint" "InverterCom:IHDM1008BCEV2R2M20"
 			(at 104.14 191.44 0)
 			(effects
@@
 			)
 		)
-		(property "Footprint" "IHDM1008BCEV2R2M20"
+		(property "Footprint" "InverterCom:IHDM1008BCEV2R2M20"
 			(at 81.28 181.28 0)
 			(effects
@@
 			)
 		)
-		(property "Footprint" "1210"
+		(property "Footprint" "Capacitor_SMD:C_1210_3225Metric_Pad1.33x2.70mm_HandSolder"
 			(at 218.1352 39.37 0)
 			(effects
@@
 			)
 		)
-		(property "Footprint" "SOIC127P600X175-8N"
+		(property "Footprint" "InverterCom:SOIC127P600X175-8N"
 			(at 212.09 136.83 0)
 			(effects
@@
 			)
 		)
-		(property "Footprint" "BEADC1608X100N"
+		(property "Footprint" "InverterCom:BEADC1608X100N"
 			(at 152.4 122.428 90)
 			(effects
@@
 			)
 		)
-		(property "Footprint" "1210"
+		(property "Footprint" "Capacitor_SMD:C_1210_3225Metric_Pad1.33x2.70mm_HandSolder"
 			(at 172.4152 86.36 0)
 			(effects
@@
 			)
 		)
-		(property "Footprint" "IHDM1008BCEV2R2M20"
+		(property "Footprint" "InverterCom:IHDM1008BCEV2R2M20"
 			(at 81.28 191.44 0)
 			(effects
@@
 			)
 		)
-		(property "Footprint" ""
+		(property "Footprint" "InverterCom:TO127P1500X470-8N-2-V1"
 			(at 115.57 118.11 0)
 			(effects
@@
 			)
 		)
-		(property "Footprint" "BEADC1608X100N"
+		(property "Footprint" "InverterCom:BEADC1608X100N"
 			(at 92.71 122.428 90)
 			(effects
@@
 			)
 		)
-		(property "Footprint" "1210"
+		(property "Footprint" "Capacitor_SMD:C_1210_3225Metric_Pad1.33x2.70mm_HandSolder"
 			(at 153.3652 59.69 0)
 			(effects
@@
 			)
 		)
-		(property "Footprint" "1210"
+		(property "Footprint" "Capacitor_SMD:C_1210_3225Metric_Pad1.33x2.70mm_HandSolder"
 			(at 230.8352 39.37 0)
 			(effects
@@
 			)
 		)
-		(property "Footprint" "VS30CDU06HM3I"
+		(property "Footprint" "InverterCom:VS30CDU06HM3I"
 			(at 49.53 54.61 0)
 			(effects
@@
 			)
 		)
-		(property "Footprint" "1210"
+		(property "Footprint" "Capacitor_SMD:C_1210_3225Metric_Pad1.33x2.70mm_HandSolder"
 			(at 140.6652 59.69 0)
 			(effects
@@
 			)
 		)
-		(property "Footprint" "IHDM1008BCEV2R2M20"
+		(property "Footprint" "InverterCom:IHDM1008BCEV2R2M20"
 			(at 104.14 181.28 0)
 			(effects
@@
 			)
 		)
-		(property "Footprint" "1210"
+		(property "Footprint" "Resistor_SMD:R_1210_3225Metric_Pad1.30x2.65mm_HandSolder"
 			(at 139.192 125.73 90)
 			(effects
@@
 			)
 		)
-		(property "Footprint" "VS30CDU06HM3I"
+		(property "Footprint" "InverterCom:VS30CDU06HM3I"
 			(at 251.46 82.55 0)
 			(effects
@@
 			)
 		)
-		(property "Footprint" "1210"
+		(property "Footprint" "Resistor_SMD:R_1210_3225Metric_Pad1.30x2.65mm_HandSolder"
 			(at 166.37 79.248 90)
 			(effects
@@
 			)
 		)
-		(property "Footprint" "VS30CDU06HM3I"
+		(property "Footprint" "InverterCom:VS30CDU06HM3I"
 			(at 251.46 68.58 0)
 			(effects
@@
 			)
 		)
-		(property "Footprint" "1210"
+		(property "Footprint" "Resistor_SMD:R_1210_3225Metric_Pad1.30x2.65mm_HandSolder"
 			(at 79.502 125.73 90)
 			(effects
@@
 			)
 		)
-		(property "Footprint" "VS30CDU06HM3I"
+		(property "Footprint" "InverterCom:VS30CDU06HM3I"
 			(at 49.53 82.55 0)
 			(effects
@@
 			)
 		)
-		(property "Footprint" ""
+		(property "Footprint" "InverterCom:TO127P1500X470-8N-2-V1"
 			(at 175.26 118.11 0)
 			(effects
@@
 			)
 		)
-		(property "Footprint" "VS30CDU06HM3I"
+		(property "Footprint" "InverterCom:VS30CDU06HM3I"
 			(at 49.53 40.64 0)
 			(effects
@@
 			)
 		)
-		(property "Footprint" "VS30CDU06HM3I"
+		(property "Footprint" "InverterCom:VS30CDU06HM3I"
 			(at 251.46 124.46 0)
 			(effects
@@
 			)
 		)
-		(property "Footprint" "IHDM1008BCEV2R2M20"
+		(property "Footprint" "InverterCom:IHDM1008BCEV2R2M20"
 			(at 104.14 171.12 0)
 			(effects
@@
 			)
 		)
-		(property "Footprint" "IHDM1008BCEV2R2M20"
+		(property "Footprint" "InverterCom:IHDM1008BCEV2R2M20"
 			(at 81.28 171.12 0)
 			(effects
@@
 			)
 		)
-		(property "Footprint" "VS30CDU06HM3I"
+		(property "Footprint" "InverterCom:VS30CDU06HM3I"
 			(at 251.46 110.49 0)
 			(effects
@@
 			)
 		)
-		(property "Footprint" "VS30CDU06HM3I"
+		(property "Footprint" "InverterCom:VS30CDU06HM3I"
 			(at 251.46 96.52 0)
 			(effects
@@
 			)
 		)
-		(property "Footprint" "1210"
+		(property "Footprint" "Resistor_SMD:R_1210_3225Metric_Pad1.30x2.65mm_HandSolder"
 			(at 139.192 137.16 90)
 			(effects
@@
 			)
 		)
-		(property "Footprint" "VS30CDU06HM3I"
+		(property "Footprint" "InverterCom:VS30CDU06HM3I"
 			(at 49.53 68.58 0)
 			(effects
@@
 			)
 		)
-		(property "Footprint" "1210"
+		(property "Footprint" "Capacitor_SMD:C_1210_3225Metric_Pad1.33x2.70mm_HandSolder"
 			(at 155.2448 121.92 0)
 			(effects
@@
 			)
 		)
-		(property "Footprint" "1210"
+		(property "Footprint" "Resistor_SMD:R_1210_3225Metric_Pad1.30x2.65mm_HandSolder"
 			(at 79.502 137.16 90)
 			(effects
@@
 			)
 		)
-		(property "Footprint" "VS30CDU06HM3I"
+		(property "Footprint" "InverterCom:VS30CDU06HM3I"
 			(at 251.46 138.43 0)
 			(effects
