File: DynamicBrakeGrid/KiCad/DynamicBrakeGrid/PowerStage.kicad_sch (KiCad schematic)
At the start: 34 parts, among them IC3 UCC27424QDRQ1, IC8 LM358DR, Q1 STWA75N60M6, Q2 STWA75N60M6, U6 ACS758xCB-200U-PFF

Commit message: Update Schematics, Inverter, Gate Driver, Mechanical, Software
Parts:
- added C39, C40: 100nF, Capacitor_SMD:C_1210_3225Metric_Pad1.33x2.70mm_HandSolder, symbol Device:C
- added R53, R54: 58, Resistor_SMD:R_1210_3225Metric_Pad1.30x2.65mm_HandSolder, symbol Device:R
Connections:
- net DC_LINK_V+: now also C12.1, C13.1, C14.1, C15.1; no longer C12.2, C13.2, C14.2, C15.2
- net GNDPWR: now also C12.2, C13.2, C14.2, C15.2; no longer C12.1, C13.1, C14.1, C15.1
- net at C47.1, R55.2, R56.1: now also C40.1
- net at C38.2, FB1.2: now also C39.2, R53.1; no longer Q1.1 (G)
- net at C47.2, FB3.2: now also C40.2, R54.1; no longer Q2.1 (G)
- net at C38.1, R51.2, R52.1: now also C39.1
- new net: Q2.1 (G), R54.2
- new net: Q1.1 (G), R53.2
Other:
- moved on the sheet: C12, C13, C14, C15
