File: Inverter/GateDriver/Connectors.kicad_sch (KiCad schematic)
At the start: 9 parts, among them J1 1548129, J2 DE09-PA-M1, J3 1548129, J5 1987724, J6 1987724, J7 1987724

Commit message: u
Parts:
- removed H1, H2, H3: MountingHole_Pad_MP, symbol Mechanical:MountingHole_Pad_MP
- removed J2: DE09-PA-M1, InverterCom:DE09PAM1, symbol InverterCom:DE09-PA-M1
- added H4, H5, H6: MountingHole_Pad_MP, MountingHole:MountingHole_5.3mm_M5_Pad, symbol Mechanical:MountingHole_Pad_MP
- added J4: 5-106505-2, 5-106505-2_3, symbol InverterCom:5-106505-2
- added Q1: ~, InverterCom:CM600HA-24H-Gate, symbol InverterCom:CM600HA-24H-Gate
- J1, J3: footprint 1548129 -> InverterCom:1548129
- J5, J6, J7: footprint 1987724 -> InverterCom:1987724; now not fitted
Connections:
- net +12V: now also J4.1
- net FAULT: now also J4.5
- net GATE_DRIVE+: now also J4.3
- net GATE_DRIVE-: now also J4.4
- net GND: now also J4.10, J4.11, J4.2
- net IGBT_COLLECTOR: now also Q1.1 (C)
- net IGBT_EMITTER: now also Q1.2 (E)
- net IGBT_GATE: now also Q1.3 (G)
- net SDI: now also J4.6
- net SDO: now also J4.7
- net SPI_CLK: now also J4.8
- net SPI_CS: now also J4.9
