File: Inverter/GateDriver/PowerSupply.kicad_sch (KiCad schematic)
At the start: 35 parts

Commit message: u
Parts:
- PS1: footprint RKE1205SH -> InverterCom:RKE1205SH
- PS4: footprint RFMM0505S -> InverterCom:RFMM0505S
Changed lines of the file:
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@@
 			)
 		)
-		(property "Footprint" "RKE1205SH"
+		(property "Footprint" "InverterCom:RKE1205SH"
 			(at 96.52 121.59 0)
 			(effects
@@
 			)
 		)
-		(property "Footprint" "RFMM0505S"
+		(property "Footprint" "InverterCom:RFMM0505S"
 			(at 59.69 202.87 0)
 			(effects
