File: Inverter/GateDriver/GateDriver.kicad_pcb (KiCad board)
At the start: 2 copper layers, 80 x 120 mm, 0 parts

Commit message: u
Parts:
- added C20: 1uF, Capacitor_SMD:C_1210_3225Metric_Pad1.33x2.70mm_HandSolder, F.Cu at (142.5, 115.9)
- added C26: 1uF, Capacitor_SMD:C_1210_3225Metric_Pad1.33x2.70mm_HandSolder, B.Cu at (148.0, 97.5)
- added C27: 100nF, Capacitor_SMD:C_1210_3225Metric_Pad1.33x2.70mm_HandSolder, B.Cu at (148.0, 102.0)
- added C28: 10uF, Capacitor_SMD:C_1210_3225Metric_Pad1.33x2.70mm_HandSolder, F.Cu at (122.5, 143.5)
- added C29: 1uF, Capacitor_SMD:C_1210_3225Metric_Pad1.33x2.70mm_HandSolder, F.Cu at (127.0, 143.5)
- added C30: 100nF, Capacitor_SMD:C_1210_3225Metric_Pad1.33x2.70mm_HandSolder, F.Cu at (131.5, 143.5)
- added C31: 10uF, Capacitor_SMD:C_1210_3225Metric_Pad1.33x2.70mm_HandSolder, F.Cu at (130.5, 124.0)
- added C32: 1uF, Capacitor_SMD:C_1210_3225Metric_Pad1.33x2.70mm_HandSolder, F.Cu at (130.4, 133.0)
- added C33: 100nF, Capacitor_SMD:C_1210_3225Metric_Pad1.33x2.70mm_HandSolder, F.Cu at (130.5, 128.5)
- added C34: 10uF, Capacitor_SMD:C_1210_3225Metric_Pad1.33x2.70mm_HandSolder, F.Cu at (85.0, 101.0)
- added C35: 1uF, Capacitor_SMD:C_1210_3225Metric_Pad1.33x2.70mm_HandSolder, F.Cu at (85.0, 96.0)
- added C36: 100nF, Capacitor_SMD:C_1210_3225Metric_Pad1.33x2.70mm_HandSolder, F.Cu at (84.0, 91.0)
- added C37: UVY1E102MPD1TD, InverterCom:CAPPRD500W60D1025H1750, B.Cu at (131.0, 152.5)
- added C38: UVY1E102MPD1TD, InverterCom:CAPPRD500W60D1025H1750, B.Cu at (154.0, 153.0)
- added C39: UVY1E102MPD1TD, InverterCom:CAPPRD500W60D1025H1750, B.Cu at (142.5, 153.0)
- added C40: UVY1E102MPD1TD, InverterCom:CAPPRD500W60D1025H1750, B.Cu at (111.0, 101.5)
- added C41: UVY1E102MPD1TD, InverterCom:CAPPRD500W60D1025H1750, B.Cu at (120.5, 96.5)
- added C42: UVY1E102MPD1TD, InverterCom:CAPPRD500W60D1025H1750, B.Cu at (111.0, 90.0)
- added C43: 10uF, Capacitor_SMD:C_1210_3225Metric_Pad1.33x2.70mm_HandSolder, F.Cu at (104.9, 93.0)
- added C44: 1uF, Capacitor_SMD:C_1210_3225Metric_Pad1.33x2.70mm_HandSolder, F.Cu at (104.9, 88.5)
- added C45: 100nF, Capacitor_SMD:C_1210_3225Metric_Pad1.33x2.70mm_HandSolder, F.Cu at (104.9, 84.0)
- added C46: UVY1E102MPD1TD, InverterCom:CAPPRD500W60D1025H1750, B.Cu at (96.6, 152.5)
- added C47: UVY1E102MPD1TD, InverterCom:CAPPRD500W60D1025H1750, B.Cu at (108.0, 152.5)
- added C48: UVY1E102MPD1TD, InverterCom:CAPPRD500W60D1025H1750, B.Cu at (119.5, 152.5)
- added C49: 10uF, Capacitor_SMD:C_1210_3225Metric_Pad1.33x2.70mm_HandSolder, F.Cu at (86.0, 132.0)
- added C50: 1uF, Capacitor_SMD:C_1210_3225Metric_Pad1.33x2.70mm_HandSolder, F.Cu at (86.0, 127.0)
- added C51: 100nF, Capacitor_SMD:C_1210_3225Metric_Pad1.33x2.70mm_HandSolder, F.Cu at (85.0, 122.0)
- added C52: 100nF, Capacitor_SMD:C_1210_3225Metric_Pad1.33x2.70mm_HandSolder, F.Cu at (104.5, 115.0)
- added C53: 1uF, Capacitor_SMD:C_1210_3225Metric_Pad1.33x2.70mm_HandSolder, F.Cu at (104.5, 119.5)
- added C54: 10uF, Capacitor_SMD:C_1210_3225Metric_Pad1.33x2.70mm_HandSolder, F.Cu at (104.5, 124.5)
- added C55: UVY1E102MPD1TD, InverterCom:CAPPRD500W60D1025H1750, B.Cu at (111.0, 133.0)
- added C56: UVY1E102MPD1TD, InverterCom:CAPPRD500W60D1025H1750, B.Cu at (111.0, 121.5)
- added C57: UVY1E102MPD1TD, InverterCom:CAPPRD500W60D1025H1750, B.Cu at (119.0, 114.5)
- added C58: 1uF, Capacitor_SMD:C_1210_3225Metric_Pad1.33x2.70mm_HandSolder, B.Cu at (161.5, 99.0)
- added C59: 1uF, Capacitor_SMD:C_1210_3225Metric_Pad1.33x2.70mm_HandSolder, F.Cu at (161.0, 99.0)
- added C60: 100nF, Capacitor_SMD:C_1210_3225Metric_Pad1.33x2.70mm_HandSolder, F.Cu at (161.0, 94.5)
- added C61: 100nF, Capacitor_SMD:C_1210_3225Metric_Pad1.33x2.70mm_HandSolder, B.Cu at (157.0, 99.0)
- added C62: 10uF, Capacitor_SMD:C_1210_3225Metric_Pad1.33x2.70mm_HandSolder, B.Cu at (148.0, 93.0)
- added C64: 100nF, Capacitor_SMD:C_1210_3225Metric_Pad1.33x2.70mm_HandSolder, F.Cu at (147.0, 115.9)
- added C65: 10pF, Capacitor_SMD:C_1210_3225Metric_Pad1.33x2.70mm_HandSolder, F.Cu at (168.0, 124.5)
- added C66: 10pF, Capacitor_SMD:C_1210_3225Metric_Pad1.33x2.70mm_HandSolder, F.Cu at (162.5, 124.5)
- added C67: 10pF, Capacitor_SMD:C_1210_3225Metric_Pad1.33x2.70mm_HandSolder, F.Cu at (157.0, 124.5)
- added C68: 10pF, Capacitor_SMD:C_1210_3225Metric_Pad1.33x2.70mm_HandSolder, F.Cu at (151.5, 124.5)
- added C69: 10pF, Capacitor_SMD:C_1210_3225Metric_Pad1.33x2.70mm_HandSolder, F.Cu at (146.0, 124.5)
- added C70: 10pF, Capacitor_SMD:C_1210_3225Metric_Pad1.33x2.70mm_HandSolder, F.Cu at (140.5, 124.5)
- added C71: 100pF, Capacitor_SMD:C_1210_3225Metric_Pad1.33x2.70mm_HandSolder, F.Cu at (168.0, 129.0)
- added C72: 100pF, Capacitor_SMD:C_1210_3225Metric_Pad1.33x2.70mm_HandSolder, F.Cu at (162.5, 129.0)
- added C73: 100pF, Capacitor_SMD:C_1210_3225Metric_Pad1.33x2.70mm_HandSolder, F.Cu at (157.0, 129.0)
- added C74: 100pF, Capacitor_SMD:C_1210_3225Metric_Pad1.33x2.70mm_HandSolder, F.Cu at (151.5, 129.0)
- added C75: 100pF, Capacitor_SMD:C_1210_3225Metric_Pad1.33x2.70mm_HandSolder, F.Cu at (146.0, 129.0)
- added C76: 100pF, Capacitor_SMD:C_1210_3225Metric_Pad1.33x2.70mm_HandSolder, F.Cu at (140.5, 129.0)
- added C77: 100pF, Capacitor_SMD:C_1210_3225Metric_Pad1.33x2.70mm_HandSolder, B.Cu at (151.6, 123.0)
- added C79: 100nF, Capacitor_SMD:C_1210_3225Metric_Pad1.33x2.70mm_HandSolder, F.Cu at (155.0, 94.5)
- added C80: 1uF, Capacitor_SMD:C_1210_3225Metric_Pad1.33x2.70mm_HandSolder, F.Cu at (155.0, 99.0)
- added C81: 100pF, Capacitor_SMD:C_1210_3225Metric_Pad1.33x2.70mm_HandSolder, F.Cu at (133.0, 89.4)
- added C82: 10nF, Capacitor_SMD:C_1210_3225Metric_Pad1.33x2.70mm_HandSolder, B.Cu at (171.5, 103.0)
- added C83: 100nF, Capacitor_SMD:C_1210_3225Metric_Pad1.33x2.70mm_HandSolder, F.Cu at (164.1, 60.0)
- added C84: 10nF, Capacitor_SMD:C_1210_3225Metric_Pad1.33x2.70mm_HandSolder, B.Cu at (171.5, 88.5)
- added C85: 10nF, Capacitor_SMD:C_1210_3225Metric_Pad1.33x2.70mm_HandSolder, F.Cu at (147.9, 102.0)
- added D10: VS-30CDU06HM3_I, InverterCom:VS30CDU06HM3I, F.Cu at (121.5, 70.0)
- added D11: VS-30CDU06HM3_I, InverterCom:VS30CDU06HM3I, F.Cu at (107.5, 69.8)
- added D12: MBRA340T3G, InverterCom:DIOM5226X220N, F.Cu at (142.5, 96.0)
- added D8: BAT54WS-7-F, InverterCom:SOD2513X120N, F.Cu at (148.0, 93.0)
- added D9: BAT54WS-7-F, InverterCom:SOD2513X120N, F.Cu at (133.0, 86.0)
- added H4: MountingHole_Pad_MP, MountingHole:MountingHole_5.3mm_M5_Pad, F.Cu at (82.5, 152.5)
- added H5: MountingHole_Pad_MP, MountingHole:MountingHole_5.3mm_M5_Pad, F.Cu at (180.0, 152.5)
- added H6: MountingHole_Pad_MP, MountingHole:MountingHole_5.3mm_M5_Pad, F.Cu at (82.5, 47.5)
- added J1: 1548129, InverterCom:1548129, F.Cu at (182.0, 89.8)
- added J3: 1548129, InverterCom:1548129, F.Cu at (182.0, 108.1)
- added J4: 5-106505-2, InverterCom:5-106505-2_3, B.Cu at (185.4, 146.4)
- added J5: 1987724, InverterCom:1987724, F.Cu at (179.0, 70.0)
- added J6: 1987724, InverterCom:1987724, F.Cu at (155.0, 59.0)
- added J7: 1987724, InverterCom:1987724, F.Cu at (112.5, 49.0)
- added PS1: RKE-1205S_H, InverterCom:RKE1205SH, B.Cu at (134.4, 141.3)
- added PS2: REC10K-2415SAW_H2, InverterCom:REC10K-AW, B.Cu at (90.2, 94.0)
- added PS3: REC10K-2409SAW_H2, InverterCom:REC10K-AW, B.Cu at (90.2, 125.0)
- added PS4: RFMM-0505S, InverterCom:RFMM0505S, B.Cu at (134.5, 119.3)
- added Q1: ~, InverterCom:CM600HA-24H-Gate, F.Cu at (178.8, 56.0)
- added R23: 47k, Resistor_SMD:R_1210_3225Metric_Pad1.30x2.65mm_HandSolder, B.Cu at (146.6, 119.5)
- added R24: 0, Resistor_SMD:R_1210_3225Metric_Pad1.30x2.65mm_HandSolder, F.Cu at (96.5, 125.0)
- added R25: 100, Resistor_SMD:R_1210_3225Metric_Pad1.30x2.65mm_HandSolder, F.Cu at (139.5, 134.6)
- added R26: 100, Resistor_SMD:R_1210_3225Metric_Pad1.30x2.65mm_HandSolder, F.Cu at (145.0, 134.5)
- added R27: 100, Resistor_SMD:R_1210_3225Metric_Pad1.30x2.65mm_HandSolder, F.Cu at (150.5, 134.5)
- added R28: 100, Resistor_SMD:R_1210_3225Metric_Pad1.30x2.65mm_HandSolder, F.Cu at (156.0, 134.5)
- added R29: 100, Resistor_SMD:R_1210_3225Metric_Pad1.30x2.65mm_HandSolder, F.Cu at (161.5, 134.6)
- added R30: 100, Resistor_SMD:R_1210_3225Metric_Pad1.30x2.65mm_HandSolder, F.Cu at (167.0, 134.5)
- added R31: 100, Resistor_SMD:R_1210_3225Metric_Pad1.30x2.65mm_HandSolder, B.Cu at (151.6, 119.5)
- added R32: 4.7, Resistor_SMD:R_1210_3225Metric_Pad1.30x2.65mm_HandSolder, F.Cu at (159.5, 80.5)
- added R33: 4.7, Resistor_SMD:R_1210_3225Metric_Pad1.30x2.65mm_HandSolder, F.Cu at (159.5, 84.7)
- added R34: 4.7, Resistor_SMD:R_1210_3225Metric_Pad1.30x2.65mm_HandSolder, F.Cu at (165.0, 84.7)
- added R35: 4.7, Resistor_SMD:R_1210_3225Metric_Pad1.30x2.65mm_HandSolder, F.Cu at (165.0, 80.5)
- added R36: 0, Resistor_SMD:R_1210_3225Metric_Pad1.30x2.65mm_HandSolder, B.Cu at (169.0, 93.0)
- added R37: 10k, Resistor_SMD:R_1210_3225Metric_Pad1.30x2.65mm_HandSolder, B.Cu at (173.5, 93.0)
- added R38: 10k, Resistor_SMD:R_1210_3225Metric_Pad1.30x2.65mm_HandSolder, B.Cu at (169.0, 107.5)
- added R39: 8.2, Resistor_SMD:R_1210_3225Metric_Pad1.30x2.65mm_HandSolder, F.Cu at (154.0, 85.0)
- added R40: 8.2, Resistor_SMD:R_1210_3225Metric_Pad1.30x2.65mm_HandSolder, F.Cu at (154.0, 80.5)
- added R41: 8.2, Resistor_SMD:R_1210_3225Metric_Pad1.30x2.65mm_HandSolder, F.Cu at (148.5, 85.0)
- added R42: 8.2, Resistor_SMD:R_1210_3225Metric_Pad1.30x2.65mm_HandSolder, F.Cu at (148.5, 80.5)
- added R43: 0, Resistor_SMD:R_1210_3225Metric_Pad1.30x2.65mm_HandSolder, B.Cu at (173.5, 107.5)
- added R44: 10k, Resistor_SMD:R_1210_3225Metric_Pad1.30x2.65mm_HandSolder, F.Cu at (164.1, 54.0)
- added R45: 33, Resistor_SMD:R_1210_3225Metric_Pad1.30x2.65mm_HandSolder, F.Cu at (148.0, 96.0)
- added R46: 1k, Resistor_SMD:R_1210_3225Metric_Pad1.30x2.65mm_HandSolder, F.Cu at (126.0, 81.0)
- added TP3: TestPoint, TestPoint:TestPoint_Loop_D2.54mm_Drill1.5mm_Beaded, F.Cu at (140.5, 104.0)
- added TP4: TestPoint, TestPoint:TestPoint_Loop_D2.54mm_Drill1.5mm_Beaded, F.Cu at (168.5, 65.0)
- added TP5: TestPoint, TestPoint:TestPoint_Loop_D2.54mm_Drill1.5mm_Beaded, F.Cu at (165.0, 91.5)
- added TP6: TestPoint, TestPoint:TestPoint_Loop_D2.54mm_Drill1.5mm_Beaded, F.Cu at (167.0, 100.0)
- added TP7: TestPoint, TestPoint:TestPoint_Loop_D2.54mm_Drill1.5mm_Beaded, F.Cu at (138.5, 94.5)
- added TP8: TestPoint, TestPoint:TestPoint_Loop_D2.54mm_Drill1.5mm_Beaded, F.Cu at (128.0, 86.0)
- added U2: PUCC5880QDFCQ1, InverterCom:SSOP32_DFC_TEX-M, F.Cu at (156.0, 108.5)
Routing:
- net IGBT_EMITTER: track 0.00 -> 75.8 mm
- net IGBT_GATE: track 0.00 -> 66.0 mm
- net IGBT_COLLECTOR: track 0.00 -> 63.5 mm
- net GATE_DRIVE-: track 0.00 -> 62.8 mm, vias 0 -> 1
- net +12V: track 0.00 -> 52.6 mm, vias 0 -> 1
- net DESAT: track 0.00 -> 50.1 mm, vias 0 -> 2
- net +5V: track 0.00 -> 47.8 mm, vias 0 -> 1
- net GATE_DRIVE+: track 0.00 -> 44.6 mm, vias 0 -> 1
- net SPI_CLK: track 0.00 -> 42.9 mm, vias 0 -> 1
- net SPI_CS: track 0.00 -> 42.7 mm, vias 0 -> 1
- net ISO_GATE_DRIVE_+15V: track 0.00 -> 37.2 mm
- net FILTERED_GATE_DRIVE-: track 0.00 -> 37.1 mm
- net FILTERED_GATE_DRIVE+: track 0.00 -> 32.3 mm
- net FAULT: track 0.00 -> 30.9 mm
- net FILTERED_SPI_CLK: track 0.00 -> 27.2 mm
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- added copper zone on B.Cu, net +12V
- added copper zone on B.Cu, net GND
- added copper zone on F.Cu, net GND
- added copper zone on B.Cu, net IGBT_EMITTER
- added copper zone on F.Cu, net IGBT_EMITTER
- added copper zone on In1.Cu, net ISO_GATE_DRIVE_+15V
- added copper zone on In2.Cu, net ISO_GATE_DRIVE_-9V
Other:
- board size 80 x 120 mm -> 112.5 x 120 mm
- copper layers 2 -> 4

Commit message: vsense
Parts:
- moved R24 34.4 mm to (102.0, 91.0), turned to 180 degrees
- moved PS3 29.8 mm to (97.2, 96.0)
- moved C54 28.6 mm to (102.0, 96.0)
- moved C49 28.3 mm to (82.0, 104.0), turned to 0 degrees
- moved C50 28.3 mm to (82.0, 99.0), turned to 0 degrees
- moved C51 28.1 mm to (83.0, 94.0), turned to 0 degrees
- moved C43 27.1 mm to (103.0, 66.0), turned to 0 degrees
- moved PS2 26.9 mm to (97.2, 68.0)
- moved C44 26.1 mm to (103.0, 62.5), turned to 0 degrees
- moved C45 26.1 mm to (103.0, 58.0), turned to 0 degrees
- moved C34 25.2 mm to (82.0, 76.0), turned to 0 degrees
- moved C35 25.2 mm to (82.0, 71.0), turned to 0 degrees
- moved C36 25.0 mm to (83.0, 66.0), turned to 0 degrees
- moved C53 18.7 mm to (102.0, 101.0)
- moved J1 18.3 mm to (182.0, 108.1)
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Routing:
- net IGBT_EMITTER: track 75.8 -> 220.8 mm, vias 0 -> 132
- net ISO_GATE_DRIVE_+15V: track 37.2 -> 139.5 mm, vias 0 -> 5
- net IGBT_GATE: track 66.0 -> 140.4 mm
- net +5VP: track 0.00 -> 73.2 mm
- net ISO_GATE_DRIVE_-9V: track 19.5 -> 85.5 mm, vias 0 -> 3
- net Net-(U2-OUTH1): track 0.00 -> 29.0 mm, vias 0 -> 2
- net Net-(U2-OUTH2): track 0.00 -> 27.2 mm, vias 0 -> 2
- net ANALOG_SENSE_2: track 0.00 -> 25.0 mm, vias 0 -> 2
- net ANALOG_SENSE_1: track 0.00 -> 24.5 mm, vias 0 -> 2
- net +12V: track 52.6 -> 74.4 mm, vias 1 -> 4
- net IGBT_COLLECTOR: track 63.5 -> 48.2 mm
- net ANALOG_INPUT_2: track 0.00 -> 15.3 mm
- net ANALOG_INPUT_1: track 0.00 -> 12.9 mm
- net GND: track 10.1 -> 17.7 mm, vias 0 -> 452
- net Net-(U2-VREF): track 0.00 -> 7.11 mm, vias 0 -> 1
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- added copper zone on In1.Cu, net GND
- added copper zone on In2.Cu, net GND
- added copper zone on In2.Cu, net IGBT_EMITTER

Commit message: Update
Parts:
- added G***: LOGO, InverterCom:Silkscreen_Logo_CelstialBeing_S, F.Cu at (110.0, 142.5)
- added G***: LOGO, InverterCom:Silkscreen_Logo_CelstialBeing_S, B.Cu at (154.5, 140.0)
- added REF**: ESD-Logo_13.2x12mm_SilkScreen, Symbol:ESD-Logo_13.2x12mm_SilkScreen, B.Cu at (87.0, 137.5)
- added REF**: KiCad-Logo2_8mm_SilkScreen, Symbol:KiCad-Logo2_8mm_SilkScreen, B.Cu at (106.5, 139.5)
- added REF**: OSHW-Logo2_14.6x12mm_SilkScreen, Symbol:OSHW-Logo2_14.6x12mm_SilkScreen, B.Cu at (86.0, 122.5)
- added REF**: WEEE-Logo_8.4x12mm_SilkScreen, Symbol:WEEE-Logo_8.4x12mm_SilkScreen, B.Cu at (122.5, 140.5)
- moved J1 2.00 mm to (180.0, 108.1)
- moved J3 2.00 mm to (180.0, 89.8)
Routing:
- net IGBT_EMITTER: track 220.8 -> 216.2 mm
- net ANALOG_INPUT_1: track 12.9 -> 10.9 mm
- net ANALOG_INPUT_2: track 15.3 -> 14.0 mm
- net +5VP: track 73.2 -> 74.0 mm
Other:
- board text added: "A_IN1 | GND | +5V"
- board text added: "A_IN2 | GND | +5V"
- board text added: "SERIAL NUMBER"
- board text added: "TO MAIN CONTROL BOARD (P/N: 56TYH)"
