File: IsolatedVoltageSensor/IsolatedVoltageSensor/Connectors.kicad_sch (KiCad schematic)
At the start: 6 parts, among them J1 Conn_01x10_Pin, J2 Conn_01x10_Pin

Commit message: finish vsense
Connections:
- net DC_LINK_BUS_ISOLATED_VSENSE: now also J2.3 (Pin_3); no longer J1.2 (Pin_2)
- net DC_LINK_BUS_VSENSE: now also J1.2 (Pin_2); no longer J2.3 (Pin_3)
- net PHASE_U_ISOLATED_VSENSE: now also J2.9 (Pin_9); no longer J1.8 (Pin_8)
- net PHASE_U_VSENSE: now also J1.4 (Pin_4); no longer J2.5 (Pin_5)
- net PHASE_V_ISOLATED_VSENSE: now also J2.7 (Pin_7); no longer J1.6 (Pin_6)
- net PHASE_V_VSENSE: now also J1.6 (Pin_6); no longer J2.7 (Pin_7)
- net PHASE_W_ISOLATED_VSENSE: now also J2.5 (Pin_5); no longer J1.4 (Pin_4)
- net PHASE_W_VSENSE: now also J1.8 (Pin_8); no longer J2.9 (Pin_9)
Changed lines of the file:
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@@
 	(generator_version "9.0")
 	(paper "A4")
-	(global_label "PHASE_U_ISOLATED_VSENSE"
+	(global_label "PHASE_V_VSENSE"
+		(shape input)
+		(at 30.48 38.1 0)
+		(fields_autoplaced yes)
+		(effects
+			(font
+				(size 1.27 1.27)
+			)
+			(justify left)
+		)
+		(property "Intersheetrefs" "${INTERSHEET_REFS}"
+			(at 49.6727 38.1 0)
+			(effects
+				(font
+					(size 1.27 1.27)
+				)
+				(justify left)
+				(hide yes)
+			)
+		)
+	)
+	(global_label "PHASE_W_ISOLATED_VSENSE"
+		(shape input)
+		(at 81.28 35.56 0)
+		(fields_autoplaced yes)
+		(effects
+			(font
+				(size 1.27 1.27)
+			)
+			(justify left)
+		)
+		(property "Intersheetrefs" "${INTERSHEET_REFS}"
+			(at 110.4512 35.56 0)
+			(effects
+				(font
+					(size 1.27 1.27)
+				)
+				(justify left)
+				(hide yes)
+			)
+		)
+	)
+	(global_label "PHASE_W_VSENSE"
 		(shape input)
 		(at 30.48 43.18 0)
@@
 		)
 		(property "Intersheetrefs" "${INTERSHEET_REFS}"
-			(at 59.5303 43.18 0)
+			(at 50.0355 43.18 0)
+			(effects
+				(font
+					(size 1.27 1.27)
+				)
+				(justify left)
+				(hide yes)
+			)
+		)
+	)
+	(global_label "PHASE_U_ISOLATED_VSENSE"
+		(shape input)
+		(at 81.28 45.72 0)
+		(fields_autoplaced yes)
+		(effects
+			(font
+				(size 1.27 1.27)
+			)
+			(justify left)
+		)
+		(property "Intersheetrefs" "${INTERSHEET_REFS}"
+			(at 110.3303 45.72 0)
+			(effects
+				(font
+					(size 1.27 1.27)
+				)
+				(justify left)
+				(hide yes)
+			)
+		)
+	)
+	(global_label "DC_LINK_BUS_VSENSE"
+		(shape input)
+		(at 30.48 27.94 0)
+		(fields_autoplaced yes)
+		(effects
+			(font
+				(size 1.27 1.27)
+			)
+			(justify left)
+		)
+		(property "Intersheetrefs" "${INTERSHEET_REFS}"
+			(at 54.0875 27.94 0)
+			(effects
+				(font
+					(size 1.27 1.27)
+				)
+				(justify left)
+				(hide yes)
+			)
+		)
+	)
+	(global_label "PHASE_V_ISOLATED_VSENSE"
+		(shape input)
+		(at 81.28 40.64 0)
+		(fields_autoplaced yes)
+		(effects
+			(font
+				(size 1.27 1.27)
+			)
+			(justify left)
+		)
+		(property "Intersheetrefs" "${INTERSHEET_REFS}"
+			(at 110.0884 40.64 0)
 			(effects
 				(font
@@
 	(global_label "DC_LINK_BUS_ISOLATED_VSENSE"
 		(shape input)
-		(at 30.48 27.94 0)
-		(fields_autoplaced yes)
-		(effects
-			(font
-				(size 1.27 1.27)
-			)
-			(justify left)
-		)
-		(property "Intersheetrefs" "${INTERSHEET_REFS}"
-			(at 63.7032 27.94 0)
-			(effects
-				(font
-					(size 1.27 1.27)
-				)
-				(justify left)
-				(hide yes)
-			)
-		)
-	)
-	(global_label "PHASE_W_VSENSE"
-		(shape input)
-		(at 81.28 45.72 0)
-		(fields_autoplaced yes)
-		(effects
-			(font
-				(size 1.27 1.27)
-			)
-			(justify left)
-		)
-		(property "Intersheetrefs" "${INTERSHEET_REFS}"
-			(at 100.8355 45.72 0)
-			(effects
-				(font
-					(size 1.27 1.27)
-				)
-				(justify left)
-				(hide yes)
-			)
-		)
-	)
-	(global_label "PHASE_V_VSENSE"
-		(shape input)
-		(at 81.28 40.64 0)
-		(fields_autoplaced yes)
-		(effects
-			(font
-				(size 1.27 1.27)
-			)
-			(justify left)
-		)
-		(property "Intersheetrefs" "${INTERSHEET_REFS}"
-			(at 100.4727 40.64 0)
-			(effects
-				(font
-					(size 1.27 1.27)
-				)
-				(justify left)
-				(hide yes)
-			)
-		)
-	)
-	(global_label "DC_LINK_BUS_VSENSE"
-		(shape input)
 		(at 81.28 30.48 0)
 		(fields_autoplaced yes)
@@
 		)
 		(property "Intersheetrefs" "${INTERSHEET_REFS}"
-			(at 104.8875 30.48 0)
+			(at 114.5032 30.48 0)
 			(effects
 				(font
@@
 	(global_label "PHASE_U_VSENSE"
 		(shape input)
-		(at 81.28 35.56 0)
-		(fields_autoplaced yes)
-		(effects
-			(font
-				(size 1.27 1.27)
-			)
-			(justify left)
-		)
-		(property "Intersheetrefs" "${INTERSHEET_REFS}"
-			(at 100.7146 35.56 0)
-			(effects
-				(font
-					(size 1.27 1.27)
-				)
-				(justify left)
-				(hide yes)
-			)
-		)
-	)
-	(global_label "PHASE_W_ISOLATED_VSENSE"
-		(shape input)
 		(at 30.48 33.02 0)
 		(fields_autoplaced yes)
@@
 		)
 		(property "Intersheetrefs" "${INTERSHEET_REFS}"
-			(at 59.6512 33.02 0)
+			(at 49.9146 33.02 0)
 			(effects
 				(font
-					(size 1.27 1.27)
-				)
-				(justify left)
-				(hide yes)
-			)
-		)
-	)
-	(global_label "PHASE_V_ISOLATED_VSENSE"
-		(shape input)
-		(at 30.48 38.1 0)
-		(fields_autoplaced yes)
-		(effects
-			(font
-				(size 1.27 1.27)
-			)
-			(justify left)
-		)
-		(property "Intersheetrefs" "${INTERSHEET_REFS}"
-			(at 59.2884 38.1 0)
-			(effects
-				(font
