File: IsolatedVoltageSensor/IsolatedVoltageSensor/IsolatedVoltageSensor.kicad_pcb (KiCad board)
At the start: 4 copper layers, 125 x 85 mm, 110 parts, among them IC1 TLV6001QDCKRQ1, IC11 TLV6001QDCKRQ1, IC12 TLV6001QDCKRQ1, IC2 TLV6001QDCKRQ1, J1 Conn_01x10_Pin, J2 Conn_01x10_Pin

Commit message: finish vsense
Parts:
- added G***: LOGO, InverterCom:Silkscreen_Logo_CelstialBeing_S, F.Cu at (192.5, 80.0)
- added G***: LOGO, InverterCom:Char_AllelujahHaptism, F.Cu at (195.0, 131.0)
- added G***: LOGO, InverterCom:Silkscreen_Logo_CelstialBeing_S, B.Cu at (177.0, 76.5)
- added REF**: OSHW-Logo2_14.6x12mm_SilkScreen, Symbol:OSHW-Logo2_14.6x12mm_SilkScreen, B.Cu at (194.0, 65.0)
- added REF**: KiCad-Logo2_8mm_SilkScreen, Symbol:KiCad-Logo2_8mm_SilkScreen, B.Cu at (161.0, 63.0)
- added REF**: WEEE-Logo_8.4x12mm_SilkScreen, Symbol:WEEE-Logo_8.4x12mm_SilkScreen, B.Cu at (145.0, 64.0)
- added REF**: ESD-Logo_13.2x12mm_SilkScreen, Symbol:ESD-Logo_13.2x12mm_SilkScreen, B.Cu at (179.0, 64.0)
- moved TP17 130.0 mm to (125.0, 77.5)
- moved TP2 122.0 mm to (125.5, 135.0)
- moved TP12 119.6 mm to (125.5, 97.0)
- moved TP7 118.2 mm to (125.5, 116.0)
- moved TP5 89.8 mm to (177.0, 140.0), turned to 90 degrees
- moved TP18 85.0 mm to (171.0, 68.0)
- moved TP13 79.2 mm to (171.5, 87.0)
- moved TP10 78.4 mm to (177.0, 120.0)
- moved TP20 78.0 mm to (177.5, 82.0)
- moved TP15 74.5 mm to (177.0, 101.0)
- moved TP3 74.0 mm to (172.0, 125.0)
- moved TP8 69.3 mm to (172.0, 105.0)
- moved TP14 59.3 mm to (196.0, 105.5)
- moved TP19 56.8 mm to (200.0, 100.0)
- moved TP9 56.0 mm to (200.5, 110.0)
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Connections:
- J1 pad 2: DC_LINK_BUS_ISOLATED_VSENSE -> DC_LINK_BUS_VSENSE
- J1 pad 4: PHASE_W_ISOLATED_VSENSE -> PHASE_U_VSENSE
- J1 pad 6: PHASE_V_ISOLATED_VSENSE -> PHASE_V_VSENSE
- J1 pad 8: PHASE_U_ISOLATED_VSENSE -> PHASE_W_VSENSE
- J2 pad 3: DC_LINK_BUS_VSENSE -> DC_LINK_BUS_ISOLATED_VSENSE
- J2 pad 5: PHASE_U_VSENSE -> PHASE_W_ISOLATED_VSENSE
- J2 pad 7: PHASE_V_VSENSE -> PHASE_V_ISOLATED_VSENSE
- J2 pad 9: PHASE_W_VSENSE -> PHASE_U_ISOLATED_VSENSE
Routing:
- net +5V: track 0.00 -> 94.7 mm, vias 0 -> 8
- net DC_LINK_BUS_VSENSE: track 0.00 -> 67.5 mm, vias 0 -> 2
- net DC_LINK_BUS_ISOLATED_VSENSE: track 0.00 -> 65.9 mm, vias 0 -> 2
- net PHASE_W_VSENSE: track 0.00 -> 57.1 mm, vias 0 -> 2
- net PHASE_W_ISOLATED_VSENSE: track 0.00 -> 56.1 mm, vias 0 -> 2
- net PHASE_U_VSENSE: track 0.00 -> 44.0 mm, vias 0 -> 2
- net PHASE_V_ISOLATED_VSENSE: track 0.00 -> 36.6 mm, vias 0 -> 2
- net PHASE_V_VSENSE: track 0.00 -> 33.0 mm, vias 0 -> 2
- net PHASE_U_ISOLATED_VSENSE: track 0.00 -> 30.4 mm, vias 0 -> 2
- net Net-(AT2-INP): track 0.00 -> 29.7 mm, vias 0 -> 2
- net Net-(AT4-INP): track 0.00 -> 29.7 mm, vias 0 -> 2
- net Net-(AT3-INP): track 0.00 -> 29.4 mm, vias 0 -> 2
- net Net-(AT1-INP): track 0.00 -> 29.3 mm, vias 0 -> 2
- net Net-(AT4-INN): track 0.00 -> 27.4 mm, vias 0 -> 2
- net Net-(AT2-INN): track 0.00 -> 27.1 mm, vias 0 -> 2
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- added copper zone on In2.Cu, net +5V
Other:
- board text added: "SERIAL NUMBER"

Commit message: Update
Changed lines of the file:
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@@
 			(psa4output no)
 			(plot_black_and_white yes)
-			(plotinvisibletext no)
 			(sketchpadsonfab no)
 			(plotpadnumbers no)
@@
 		)
 		(embedded_fonts no)
-		(model "../../../3D/TMP236A2DCKR.stp"
+		(model "../../3D/TMP236A2DCKR.stp"
 			(offset
 				(xyz 0 0 0)
@@
 		)
 		(embedded_fonts no)
-		(model "../../../3D/TMP236A2DCKR.stp"
+		(model "../../3D/TMP236A2DCKR.stp"
 			(offset
 				(xyz 0 0 0)
@@
 		(tags "Attenuator or Isolator")
 		(property "Reference" "AT1"
-			(at 0 -6.5 0)
+			(at 2.225 -6.5 0)
 			(layer "F.SilkS")
 			(effects
@@
 		)
 		(embedded_fonts no)
-		(model "AMC3330QDWERQ1.stp"
+		(model "/home/tliao/Nextcloud/TractionInverterV3/3D/AMC3330QDWERQ1.stp"
 			(offset
 				(xyz 0 0 0)
@@
 		(tags "Attenuator or Isolator")
 		(property "Reference" "AT4"
-			(at 0 -6.5 0)
+			(at 2.225 -6.5 0)
 			(layer "F.SilkS")
 			(effects
@@
 		)
 		(embedded_fonts no)
-		(model "AMC3330QDWERQ1.stp"
+		(model "/home/tliao/Nextcloud/TractionInverterV3/3D/AMC3330QDWERQ1.stp"
 			(offset
 				(xyz 0 0 0)
@@
 		)
 		(embedded_fonts no)
-		(model "../../../3D/TMP236A2DCKR.stp"
+		(model "../../3D/TMP236A2DCKR.stp"
 			(offset
 				(xyz 0 0 0)
@@
 		)
 		(embedded_fonts no)
-		(model "../../../3D/TMP236A2DCKR.stp"
+		(model "../../3D/TMP236A2DCKR.stp"
 			(offset
 				(xyz 0 0 0)
@@
 		(tags "Attenuator or Isolator")
 		(property "Reference" "AT2"
-			(at 0 -6.5 0)
+			(at 2.225 -6.5 0)
 			(layer "F.SilkS")
 			(effects
@@
 		)
 		(embedded_fonts no)
-		(model "AMC3330QDWERQ1.stp"
+		(model "/home/tliao/Nextcloud/TractionInverterV3/3D/AMC3330QDWERQ1.stp"
 			(offset
 				(xyz 0 0 0)
@@
 		(tags "Attenuator or Isolator")
 		(property "Reference" "AT3"
-			(at 0 -6.5 0)
+			(at 2.225 -6.5 0)
 			(layer "F.SilkS")
 			(effects
@@
 		)
 		(embedded_fonts no)
-		(model "AMC3330QDWERQ1.stp"
+		(model "/home/tliao/Nextcloud/TractionInverterV3/3D/AMC3330QDWERQ1.stp"
 			(offset
 				(xyz 0 0 0)
@@
 		(layer "F.SilkS")
 	)
+	(gr_line
+		(start 150 57.5)
+		(end 150 142.5)
+		(stroke
+			(width 0.3)
+			(type dash)
+		)
+		(layer "F.SilkS")
+	)
