File: PowerBoard/PowerBoard.kicad_pcb (KiCad board)
At the start: 2 copper layers, 390 x 200 mm, 160 parts, among them IC1 TLV6001QDCKRQ1, IC10 ACS772ECB-400B-PFF-T, IC11 TLV6001QDCKRQ1, IC12 TLV6001QDCKRQ1, IC2 TLV6001QDCKRQ1, IC3 ACS772ECB-400B-PFF-T, IC4 ACS772ECB-400B-PFF-T, IC5 ACS772ECB-400B-PFF-T, IC6 ACS772ECB-400B-PFF-T, IC7 ACS772ECB-400B-PFF-T, IC8 ACS772ECB-400B-PFF-T, IC9 ACS772ECB-400B-PFF-T

Commit message: vsense
Parts:
- added C100: B32774X0205K000, InverterCom:B32774X__31.5_x_12.5_, F.Cu at (224.0, 60.5)
- added C101: ALH82A750CB600, InverterCom:ALH82A750CB600, F.Cu at (133.8, -33.1)
- added C102: ALH82A750CB600, InverterCom:ALH82A750CB600, F.Cu at (166.9, -33.1)
- added C103: B32652A0104K000, InverterCom:B32652__18_x_9_, F.Cu at (237.0, 229.3)
- added C104: B32652A0104K000, InverterCom:B32652__18_x_9_, F.Cu at (281.0, 229.3)
- added C105: B32774X0205K000, InverterCom:B32774X__31.5_x_12.5_, F.Cu at (224.0, 228.6)
- added C106: ALH82A750CB600, InverterCom:ALH82A750CB600, F.Cu at (200.0, -33.1)
- added C107: ALH82A750CB600, InverterCom:ALH82A750CB600, F.Cu at (233.1, -33.1)
- added C108: B32652A0104K000, InverterCom:B32652__18_x_9_, F.Cu at (123.0, 229.3)
- added C109: B32652A0104K000, InverterCom:B32652__18_x_9_, F.Cu at (166.0, 229.3)
- added C110: B32774X0205K000, InverterCom:B32774X__31.5_x_12.5_, F.Cu at (110.0, 228.6)
- added C111: ALH82A750CB600, InverterCom:ALH82A750CB600, F.Cu at (266.2, -33.1)
- added C112: ALH82A750CB600, InverterCom:ALH82A750CB600, F.Cu at (299.3, -33.1)
- added C20: B32652A0104K000, InverterCom:B32652__18_x_9_, F.Cu at (7.00, 46.0)
- added C84: B32652A0104K000, InverterCom:B32652__18_x_9_, F.Cu at (51.0, 47.0)
- added C85: B32774X0205K000, InverterCom:B32774X__31.5_x_12.5_, F.Cu at (-6.00, 59.5)
- added C86: C4AQNBW5200M3LJ, InverterCom:C4AQNBW5200M3LJ, F.Cu at (83.3, 70.5)
- added C87: C4AQNBW5200M3LJ, InverterCom:C4AQNBW5200M3LJ, F.Cu at (83.2, 229.0)
- added C88: B32652A0104K000, InverterCom:B32652__18_x_9_, F.Cu at (51.0, 229.0)
- added C89: B32652A0104K000, InverterCom:B32652__18_x_9_, F.Cu at (7.00, 229.3)
- added C90: B32774X0205K000, InverterCom:B32774X__31.5_x_12.5_, F.Cu at (-6.00, 228.6)
- added C91: C4AQNBW5200M3LJ, InverterCom:C4AQNBW5200M3LJ, F.Cu at (198.3, 70.0)
- added C92: C4AQNBW5200M3LJ, InverterCom:C4AQNBW5200M3LJ, F.Cu at (198.3, 229.0)
- added C93: B32652A0104K000, InverterCom:B32652__18_x_9_, F.Cu at (123.0, 47.0)
- added C94: B32652A0104K000, InverterCom:B32652__18_x_9_, F.Cu at (166.0, 47.0)
- added C95: B32774X0205K000, InverterCom:B32774X__31.5_x_12.5_, F.Cu at (110.0, 60.5)
- added C96: C4AQNBW5200M3LJ, InverterCom:C4AQNBW5200M3LJ, F.Cu at (313.3, 70.5)
- added C97: C4AQNBW5200M3LJ, InverterCom:C4AQNBW5200M3LJ, F.Cu at (313.1, 229.0)
- added C98: B32652A0104K000, InverterCom:B32652__18_x_9_, F.Cu at (237.0, 47.3)
- added C99: B32652A0104K000, InverterCom:B32652__18_x_9_, F.Cu at (281.0, 47.3)
- added J1: ~, InverterCom:BusBarConnection, F.Cu at (-83.0, 242.5)
- added J2: ~, InverterCom:BusBarConnection, F.Cu at (-83.0, 72.5)
- added J3: ~, InverterCom:BusBarConnection, F.Cu at (77.0, 99.5)
- added J4: ~, InverterCom:BusBarConnection, F.Cu at (192.0, 99.5)
- added J5: ~, InverterCom:BusBarConnection, F.Cu at (307.0, 99.5)
- added PS1: RKE-1205S_H, InverterCom:RKE1205SH, F.Cu at (-20.9, 103.8)
- moved C22 576.9 mm to (-87.0, 34.0), turned to -90 degrees
- moved C21 572.0 mm to (-82.0, 31.0), turned to 90 degrees
- moved R2 561.0 mm to (-77.0, 30.0), turned to 90 degrees
- moved C34 544.3 mm to (-35.0, 46.0), turned to -90 degrees
- moved C23 520.6 mm to (-30.0, 43.0)
- moved R1 515.4 mm to (-30.0, 37.0), turned to 180 degrees
- moved IC5 515.2 mm to (53.1, 144.6)
- moved IC6 514.2 mm to (56.9, 94.6), turned to 180 degrees
- moved C25 473.6 mm to (53.0, 154.0)
- moved C19 467.2 mm to (53.0, 147.5), turned to 180 degrees
- moved C32 461.7 mm to (58.6, 90.9)
- moved R3 454.8 mm to (57.5, 148.4), turned to -90 degrees
- moved C29 453.2 mm to (59.0, 86.0)
- moved IC7 448.1 mm to (168.1, 144.6)
- moved R4 440.8 mm to (53.0, 91.0), turned to -90 degrees
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Routing:
- net +5V: track 0.00 -> 592.7 mm, vias 0 -> 6
- net GND: track 0.00 -> 570.1 mm, vias 0 -> 10
- net DC_LINK_BUS_CURRENT_SENSE: track 0.00 -> 186.6 mm, vias 0 -> 2
- net PHASE_V_ISENSE: track 0.00 -> 170.4 mm, vias 0 -> 2
- net PHASE_U_ISENSE: track 0.00 -> 148.7 mm, vias 0 -> 2
- net PHASE_W_ISENSE: track 0.00 -> 95.0 mm, vias 0 -> 2
- net Net-(IC3-VIOUT): track 0.00 -> 15.1 mm
- net Net-(IC4-VIOUT): track 0.00 -> 3.33 mm
- net Net-(IC7-VIOUT): track 0.00 -> 3.31 mm
- net Net-(IC9-VIOUT): track 0.00 -> 3.30 mm
- net Net-(IC10-VIOUT): track 0.00 -> 2.95 mm
- net Net-(IC5-VIOUT): track 0.00 -> 2.56 mm
- net Net-(IC8-VIOUT): track 0.00 -> 2.09 mm
- net Net-(IC6-VIOUT): track 0.00 -> 2.09 mm
- added copper zone on F.Cu, net DC_LINK_BUS
- added copper zone on F.Cu, net DC_LINK_BUS_IN
- added copper zone on In2.Cu, net GND
- added copper zone on B.Cu, net GNDPWR
- added copper zone on F.Cu, net GNDPWR
- added copper zone on In1.Cu, net GNDPWR
- added copper zone on In2.Cu, net GNDPWR
- added copper zone on F.Cu, net PHASE_U
- added copper zone on F.Cu, net PHASE_U_OUT
- added copper zone on F.Cu, net PHASE_V
- added copper zone on F.Cu, net PHASE_V_OUT
- added copper zone on F.Cu, net PHASE_W
- added copper zone on F.Cu, net PHASE_W_OUT
Other:
- board size 390 x 200 mm -> 410 x 320 mm
- copper layers 2 -> 4
- board text added: "DC LINK BUS +"
- board text added: "DC LINK BUS -"
- board text added: "PHASE U"
- board text added: "PHASE V"
- board text added: "PHASE W"

Commit message: Update
Parts:
- removed C35, C39, C45, C53, C54, C57, C65, C66, C69, C77, C78, C81: 1uF, Capacitor_SMD:C_1210_3225Metric_Pad1.33x2.70mm_HandSolder
- removed C36, C38, C42, C44, C47, C50, C52, C55, C58, C59, C62, C64, C67, C70, C71, C74, C76, C79, C82, C83: 100nF, Capacitor_SMD:C_1210_3225Metric_Pad1.33x2.70mm_HandSolder
- removed C40, C41, C43, C46, C48, C49, C51, C56, C60, C61, C63, C68, C72, C73, C75, C80: 10nF, Capacitor_SMD:C_1210_3225Metric_Pad1.33x2.70mm_HandSolder
- removed IC1, IC11, IC12, IC2: TLV6001QDCKRQ1, InverterCom:SOT65P210X110-5N
- removed R37, R38, R43, R44, R49, R50, R55, R56: 0, Resistor_SMD:R_1210_3225Metric_Pad1.30x2.65mm_HandSolder
- removed R39, R40, R45, R46, R51, R52, R57, R58: 10k, Resistor_SMD:R_1210_3225Metric_Pad1.30x2.65mm_HandSolder
- removed R41, R42, R47, R48, R53, R54, R59, R60: 16.5k, Resistor_SMD:R_1210_3225Metric_Pad1.30x2.65mm_HandSolder
- added G***: LOGO, InverterCom:HIGHVOLTAGE_40mm, F.Cu at (224.0, 110.0)
- added G***: LOGO, InverterCom:Char_GaelioBauduin_30mm, F.Cu at (-100.0, -9.00)
- added G***: LOGO, InverterCom:Silkscreen_Logo_CelstialBeing_S, F.Cu at (309.0, 165.0)
- added G***: LOGO, InverterCom:Silkscreen_Logo_CelstialBeing_S, B.Cu at (-104.5, 101.2)
- added H1: MountingHole_Pad, MountingHole:MountingHole_5.3mm_M5_ISO7380_Pad, F.Cu at (-94.2, 102.5)
- added H10: MountingHole_Pad, MountingHole:MountingHole_5.3mm_M5_ISO7380_Pad, F.Cu at (216.5, -21.0)
- added H11: MountingHole_Pad, MountingHole:MountingHole_5.3mm_M5_ISO7380_Pad, F.Cu at (183.5, -21.5)
- added H12: MountingHole_Pad, MountingHole:MountingHole_5.3mm_M5_ISO7380_Pad, F.Cu at (150.5, -21.5)
- added H13: MountingHole_Pad, MountingHole:MountingHole_5.3mm_M5_ISO7380_Pad, F.Cu at (117.0, -21.5)
- added H14: MountingHole_Pad, MountingHole:MountingHole_5.3mm_M5_ISO7380_Pad, F.Cu at (84.0, -21.5)
- added H15: MountingHole_Pad, MountingHole:MountingHole_5.3mm_M5_ISO7380_Pad, F.Cu at (50.5, -21.5)
- added H16: MountingHole_Pad, MountingHole:MountingHole_5.3mm_M5_ISO7380_Pad, F.Cu at (17.5, -21.5)
- added H17: MountingHole_Pad, MountingHole:MountingHole_5.3mm_M5_ISO7380_Pad, F.Cu at (-15.5, -22.0)
- added H18: MountingHole_Pad, MountingHole:MountingHole_5.3mm_M5_ISO7380_Pad, F.Cu at (-48.5, -22.0)
- added H19: MountingHole_Pad, MountingHole:MountingHole_5.3mm_M5_ISO7380_Pad, F.Cu at (-81.5, -21.5)
- added H19: MountingHole_Pad, MountingHole:MountingHole_5.3mm_M5_ISO7380_Pad, F.Cu at (-15.0, 10.0)
- added H2: MountingHole_Pad, MountingHole:MountingHole_5.3mm_M5_ISO7380_Pad, F.Cu at (-23.5, 102.5)
- added H20: MountingHole_Pad, MountingHole:MountingHole_5.3mm_M5_ISO7380_Pad, F.Cu at (117.5, 10.6)
- added H21: MountingHole_Pad, MountingHole:MountingHole_5.3mm_M5_ISO7380_Pad, F.Cu at (217.5, 10.0)
- added H22: MountingHole_Pad, MountingHole:MountingHole_5.3mm_M5_ISO7380_Pad, F.Cu at (7.00, 202.0)
- added H23: MountingHole_Pad, MountingHole:MountingHole_5.3mm_M5_ISO7380_Pad, F.Cu at (123.0, 202.0)
- added H24: MountingHole_Pad, MountingHole:MountingHole_5.3mm_M5_ISO7380_Pad, F.Cu at (237.0, 202.0)
- added H3: MountingHole_Pad, MountingHole:MountingHole_5.3mm_M5_ISO7380_Pad, F.Cu at (-93.5, 212.5)
- added H4: MountingHole_Pad, MountingHole:MountingHole_5.3mm_M5_ISO7380_Pad, F.Cu at (-23.5, 212.5)
- added H5: MountingHole_Pad, MountingHole:MountingHole_5.3mm_M5_ISO7380_Pad, F.Cu at (-100.0, -45.0)
- added H6: MountingHole_Pad, MountingHole:MountingHole_5.3mm_M5_ISO7380_Pad, F.Cu at (-100.0, 245.0)
- added H7: MountingHole_Pad, MountingHole:MountingHole_5.3mm_M5_ISO7380_Pad, F.Cu at (310.0, 245.0)
- added H8: MountingHole_Pad, MountingHole:MountingHole_5.3mm_M5_ISO7380_Pad, F.Cu at (282.5, -22.5)
- added H9: MountingHole_Pad, MountingHole:MountingHole_5.3mm_M5_ISO7380_Pad, F.Cu at (249.5, -21.5)
- added J6: L717SDB25PA4CH3R, InverterCom:L717SDB25PA4CH3R, B.Cu at (-95.0, 122.2)
- added J8: Conn_01x10_Socket, Connector_PinSocket_2.54mm:PinSocket_1x10_P2.54mm_Vertical, F.Cu at (-68.5, 215.0)
- added J9: Conn_01x10_Socket, Connector_PinSocket_2.54mm:PinSocket_1x10_P2.54mm_Vertical, F.Cu at (-68.5, 100.0)
- added LED1: LTST-C230CKT, InverterCom:LEDC3216X120N, F.Cu at (-104.0, 175.0)
- added LED2: LTST-C230GKT, InverterCom:LEDC3216X120N, F.Cu at (-104.0, 180.0)
- added LED3: LTST-C230GKT, InverterCom:LEDC3216X120N, F.Cu at (-104.0, 185.0)
- added LED4: LTST-C230GKT, InverterCom:LEDC3216X120N, F.Cu at (-104.0, 190.0)
- added R62: 220, Resistor_SMD:R_1210_3225Metric_Pad1.30x2.65mm_HandSolder, F.Cu at (-96.5, 175.0)
- added R63: 220, Resistor_SMD:R_1210_3225Metric_Pad1.30x2.65mm_HandSolder, F.Cu at (-96.5, 180.0)
- added R64: 220, Resistor_SMD:R_1210_3225Metric_Pad1.30x2.65mm_HandSolder, F.Cu at (-96.5, 185.0)
- added R65: 1k, Resistor_SMD:R_1210_3225Metric_Pad1.30x2.65mm_HandSolder, F.Cu at (-96.5, 190.0)
- added REF**: WEEE-Logo_8.4x12mm_SilkScreen, Symbol:WEEE-Logo_8.4x12mm_SilkScreen, B.Cu at (-99.3, 56.0)
- added REF**: OSHW-Logo2_14.6x12mm_SilkScreen, Symbol:OSHW-Logo2_14.6x12mm_SilkScreen, B.Cu at (-100.3, 6.97)
- added REF**: ESD-Logo_13.2x12mm_SilkScreen, Symbol:ESD-Logo_13.2x12mm_SilkScreen, B.Cu at (-99.3, 22.0)
- added REF**: KiCad-Logo2_8mm_SilkScreen, Symbol:KiCad-Logo2_8mm_SilkScreen, B.Cu at (-98.3, 40.0)
- moved R36 587.7 mm to (-67.5, 200.0)
- moved R29 577.3 mm to (-67.5, 190.0)
- moved R28 572.5 mm to (-61.5, 190.0)
- moved R35 568.1 mm to (-61.5, 200.0)
- moved R27 567.7 mm to (-55.5, 190.0)
- moved R22 567.4 mm to (-67.5, 180.0)
- moved R34 563.1 mm to (-55.5, 200.0)
- moved R21 562.4 mm to (-61.5, 180.0)
- moved R14 558.8 mm to (-67.5, 170.0)
- moved R33 558.2 mm to (-49.5, 200.0)
- moved R20 557.5 mm to (-55.5, 180.0)
- moved R32 553.4 mm to (-43.5, 200.0)
- moved R19 552.6 mm to (-49.4, 180.0)
- moved R15 552.2 mm to (-61.5, 170.0)
- moved R31 548.6 mm to (-37.5, 200.0)
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Routing:
- net PHASE_W_ISENSE: track 95.0 -> 490.3 mm
- net +5V: track 592.7 -> 895.0 mm, vias 6 -> 9
- net PHASE_W: track 0.00 -> 266.8 mm, vias 0 -> 1
- net PHASE_V_ISENSE: track 170.4 -> 377.2 mm, vias 2 -> 3
- net +12V: track 0.00 -> 204.8 mm, vias 0 -> 3
- net DC_LINK_BUS: track 0.00 -> 182.1 mm
- net GND: track 570.1 -> 735.2 mm, vias 10 -> 11
- net PHASE_V: track 0.00 -> 163.7 mm, vias 0 -> 2
- net PHASE_U_ISENSE: track 148.7 -> 265.5 mm, vias 2 -> 3
- net GNDPWR: track 0.00 -> 92.8 mm, vias 0 -> 4
- net PHASE_W_ISOLATED_VSENSE: track 0.00 -> 91.9 mm, vias 0 -> 1
- net PHASE_V_ISOLATED_VSENSE: track 0.00 -> 80.2 mm, vias 0 -> 1
- net DC_LINK_BUS_ISOLATED_VSENSE: track 0.00 -> 71.1 mm, vias 0 -> 1
- net PHASE_U_ISOLATED_VSENSE: track 0.00 -> 68.5 mm, vias 0 -> 1
- net DC_LINK_BUS_VSENSE: track 0.00 -> 63.1 mm, vias 0 -> 1
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- added copper zone on B.Cu, net GND
- added copper zone on F.Cu, net GND
- added copper zone on In1.Cu, net GND
Other:
- board size 410 x 320 mm -> 430 x 310 mm
- board text added: "DANGER: HAUTE TENSION"
- board text added: "GATE DRIVER COLLECTOR (U_HIGH) ->"
- board text added: "GATE DRIVER COLLECTOR (U_LOW) ATTACH WIRE TO HOLE FROM GATE DRIVER COLLECTOR"
- board text added: "GATE DRIVER COLLECTOR (V_HIGH) ->"
- board text added: "GATE DRIVER COLLECTOR (V_LOW) ATTACH WIRE TO HOLE FROM GATE DRIVER COLLECTOR"
- board text added: "GATE DRIVER COLLECTOR (W_HIGH) ->"
- board text added: "GATE DRIVER COLLECTOR (W_LOW) ATTACH WIRE TO HOLE FROM GATE DRIVER COLLECTOR"
- board text added: "SERIAL NUMBER"
- board text added: "TO CONTROL BOARD (P/N: 56TYH)"
- board text added: "ВЫСОКОЕ НАПРЯЖЕНИЕ"
- board text added: "高電圧注意"
