File: PowerBoard/CurrentSense.kicad_sch (KiCad schematic)
At the start: 16 parts, among them IC10 ACS772ECB-400B-PFF-T, IC3 ACS772ECB-400B-PFF-T, IC4 ACS772ECB-400B-PFF-T, IC5 ACS772ECB-400B-PFF-T, IC6 ACS772ECB-400B-PFF-T, IC7 ACS772ECB-400B-PFF-T, IC8 ACS772ECB-400B-PFF-T, IC9 ACS772ECB-400B-PFF-T

Commit message: u
Parts:
- added C19, C22, C24, C26, C27, C30, C32, C34: 100nF, Capacitor_SMD:C_1210_3225Metric_Pad1.33x2.70mm_HandSolder, symbol Device:C_Small
- added C21, C23, C25, C28, C29, C31, C33, C37: 1uF, Capacitor_SMD:C_1210_3225Metric_Pad1.33x2.70mm_HandSolder, symbol Device:C_Small
- R1, R2, R3, R4, R5, R6, R7, R8: footprint 1210 -> Resistor_SMD:R_1210_3225Metric_Pad1.30x2.65mm_HandSolder
Connections:
- net +5V: now also C19.2, C21.1, C22.2, C23.1, C24.2, C25.1, C26.2, C27.1, C28.1, C29.1, C30.1, C31.1, C32.1, C33.1, C34.1, C37.1
- net GND: now also C19.1, C21.2, C22.1, C23.2, C24.1, C25.2, C26.1, C27.2, C28.2, C29.2, C30.2, C31.2, C32.2, C33.2, C34.2, C37.2
- net PHASE_U_SENSE renamed PHASE_U_ISENSE
- net PHASE_V_SENSE renamed PHASE_V_ISENSE
- net PHASE_W_SENSE renamed PHASE_W_ISENSE

Commit message: Hardware updates
Parts:
- added C35, C39, C42, C45: 1nF, Capacitor_SMD:C_1210_3225Metric_Pad1.33x2.70mm_HandSolder, symbol Device:C_Small
- added C36, C40, C43, C46: 10nF, Capacitor_SMD:C_1210_3225Metric_Pad1.33x2.70mm_HandSolde, symbol Device:C_Small
- added C38, C41, C44, C47: 100nF, Capacitor_SMD:C_1210_3225Metric_Pad1.33x2.70mm_HandSolde, symbol Device:C_Small
Connections:
- net DC_LINK_BUS: now also IC4.5 (IP-); no longer IC4.4 (IP+)
- net DC_LINK_BUS_CURRENT_SENSE: now also C35.1, C36.1, C38.1
- net DC_LINK_BUS_IN: now also IC4.4 (IP+); no longer IC4.5 (IP-)
- net GND: now also C35.2, C36.2, C38.2, C39.2, C40.2, C41.2, C42.2, C43.2, C44.2, C45.2, C46.2, C47.2
- net PHASE_U: now also IC6.5 (IP-); no longer IC6.4 (IP+)
- net PHASE_U_ISENSE: now also C39.1, C40.1, C41.1
- net PHASE_U_OUT: now also IC6.4 (IP+); no longer IC6.5 (IP-)
- net PHASE_V: now also IC8.5 (IP-); no longer IC8.4 (IP+)
- net PHASE_V_ISENSE: now also C42.1, C43.1, C44.1
- net PHASE_V_OUT: now also IC8.4 (IP+); no longer IC8.5 (IP-)
- net PHASE_W: now also IC10.5 (IP-); no longer IC10.4 (IP+)
- net PHASE_W_ISENSE: now also C45.1, C46.1, C47.1
- net PHASE_W_OUT: now also IC10.4 (IP+); no longer IC10.5 (IP-)
Other:
- moved on the sheet: C23, C27, C28, C29, C30, C32, C33, C34, IC10, IC4, IC6, IC8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
