File: PowerBoard/PowerAssembly.kicad_sch (KiCad schematic)
At the start: 24 parts

Commit message: u
Parts:
- C1, C10, C11, C12, C13, C14, C15, C16, C17, C18, C2, C3, C4, C5, C6, C7, C8, C9: footprint ALH82A750CB600 -> InverterCom:ALH82A750CB600
- Q1, Q2, Q3, Q4, Q5, Q6: footprint (none) -> InverterCom:CM600HA-24H-PWR
Changed lines of the file:
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@@
 			)
 		)
-		(property "Footprint" "ALH82A750CB600"
+		(property "Footprint" "InverterCom:ALH82A750CB600"
 			(at -6.02 148.59 0)
 			(effects
@@
 			)
 		)
-		(property "Footprint" "ALH82A750CB600"
+		(property "Footprint" "InverterCom:ALH82A750CB600"
 			(at 18.11 97.79 0)
 			(effects
@@
 			)
 		)
-		(property "Footprint" "ALH82A750CB600"
+		(property "Footprint" "InverterCom:ALH82A750CB600"
 			(at 18.11 148.59 0)
 			(effects
@@
 			)
 		)
-		(property "Footprint" "ALH82A750CB600"
+		(property "Footprint" "InverterCom:ALH82A750CB600"
 			(at 42.24 148.59 0)
 			(effects
@@
 			)
 		)
-		(property "Footprint" "ALH82A750CB600"
+		(property "Footprint" "InverterCom:ALH82A750CB600"
 			(at -30.15 97.79 0)
 			(effects
@@
 			)
 		)
-		(property "Footprint" "ALH82A750CB600"
+		(property "Footprint" "InverterCom:ALH82A750CB600"
 			(at 66.37 97.79 0)
 			(effects
@@
 			)
 		)
-		(property "Footprint" ""
+		(property "Footprint" "InverterCom:CM600HA-24H-PWR"
 			(at 45.72 63.5 0)
 			(effects
@@
 			)
 		)
-		(property "Footprint" "ALH82A750CB600"
+		(property "Footprint" "InverterCom:ALH82A750CB600"
 			(at -54.28 148.59 0)
 			(effects
@@
 			)
 		)
-		(property "Footprint" ""
+		(property "Footprint" "InverterCom:CM600HA-24H-PWR"
 			(at 100.33 33.02 0)
 			(effects
@@
 			)
 		)
-		(property "Footprint" "ALH82A750CB600"
+		(property "Footprint" "InverterCom:ALH82A750CB600"
 			(at -6.02 124.46 0)
 			(effects
@@
 			)
 		)
-		(property "Footprint" ""
+		(property "Footprint" "InverterCom:CM600HA-24H-PWR"
 			(at 100.33 63.5 0)
 			(effects
@@
 			)
 		)
-		(property "Footprint" "ALH82A750CB600"
+		(property "Footprint" "InverterCom:ALH82A750CB600"
 			(at -30.15 124.46 0)
 			(effects
@@
 			)
 		)
-		(property "Footprint" "ALH82A750CB600"
+		(property "Footprint" "InverterCom:ALH82A750CB600"
 			(at 18.11 124.46 0)
 			(effects
@@
 			)
 		)
-		(property "Footprint" "ALH82A750CB600"
+		(property "Footprint" "InverterCom:ALH82A750CB600"
 			(at 42.24 97.79 0)
 			(effects
@@
 			)
 		)
-		(property "Footprint" "ALH82A750CB600"
+		(property "Footprint" "InverterCom:ALH82A750CB600"
 			(at -6.02 97.79 0)
 			(effects
@@
 			)
 		)
-		(property "Footprint" "ALH82A750CB600"
+		(property "Footprint" "InverterCom:ALH82A750CB600"
 			(at -30.15 148.59 0)
 			(effects
@@
 			)
 		)
-		(property "Footprint" "ALH82A750CB600"
+		(property "Footprint" "InverterCom:ALH82A750CB600"
 			(at -54.28 97.79 0)
 			(effects
@@
 			)
 		)
-		(property "Footprint" "ALH82A750CB600"
+		(property "Footprint" "InverterCom:ALH82A750CB600"
 			(at 66.37 148.59 0)
 			(effects
@@
 			)
 		)
-		(property "Footprint" ""
+		(property "Footprint" "InverterCom:CM600HA-24H-PWR"
 			(at 45.72 33.02 0)
 			(effects
@@
 			)
 		)
-		(property "Footprint" "ALH82A750CB600"
+		(property "Footprint" "InverterCom:ALH82A750CB600"
 			(at 66.37 124.46 0)
 			(effects
@@
 			)
 		)
-		(property "Footprint" "ALH82A750CB600"
+		(property "Footprint" "InverterCom:ALH82A750CB600"
 			(at -54.28 124.46 0)
 			(effects
@@
 			)
 		)
-		(property "Footprint" ""
+		(property "Footprint" "InverterCom:CM600HA-24H-PWR"
 			(at 73.66 33.02 0)
 			(effects
@@
 			)
 		)
-		(property "Footprint" "ALH82A750CB600"
+		(property "Footprint" "InverterCom:ALH82A750CB600"
 			(at 42.24 124.46 0)
 			(effects
@@
 			)
 		)
-		(property "Footprint" ""
+		(property "Footprint" "InverterCom:CM600HA-24H-PWR"
 			(at 73.66 63.5 0)
 			(effects

Commit message: vsense
Parts:
- added C100, C105, C110, C85, C90, C95: B32774X0205K000, InverterCom:B32774X__31.5_x_12.5_, symbol InverterCom:B32774X0205K000
- added C101, C102, C106, C107, C111, C112: ALH82A750CB600, InverterCom:ALH82A750CB600, symbol InverterCom:ALH82A750CB600
- added C103, C104, C108, C109, C20, C84, C88, C89, C93, C94, C98, C99: B32652A0104K000, InverterCom:B32652__18_x_9_, symbol InverterCom:B32652A0104K000
- added C86, C87, C91, C92, C96, C97: C4AQNBW5200M3LJ, InverterCom:C4AQNBW5200M3LJ, symbol InverterCom:C4AQNBW5200M3LJ
Connections:
- net DC_LINK_BUS: now also C100.2, C101.1, C102.1, C106.1, C107.1, C111.1, C112.1, C20.2, C84.2, C85.2, C86.2, C86.4, C91.2, C91.4, C93.2, C94.2, C95.2, C96.2, C96.4, C98.2, C99.2
- net GNDPWR: now also C101.2, C102.2, C103.1, C104.1, C105.1, C106.2, C107.2, C108.1, C109.1, C110.1, C111.2, C112.2, C87.1, C87.3, C88.1, C89.1, C90.1, C92.1, C92.3, C97.1, C97.3
- net PHASE_U: now also C20.1, C84.1, C85.1, C86.1, C86.3, C87.2, C87.4, C88.2, C89.2, C90.2
- net PHASE_V: now also C108.2, C109.2, C110.2, C91.1, C91.3, C92.2, C92.4, C93.1, C94.1, C95.1
- net PHASE_W: now also C100.1, C103.2, C104.2, C105.2, C96.1, C96.3, C97.2, C97.4, C98.1, C99.1
Other:
- moved on the sheet: Q1, Q2, Q3, Q4, Q5, Q6

Commit message: Hardware updates
Other:
- note added: "add zeners"
Changed lines of the file:
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@@
 	(generator_version "9.0")
 	(paper "A4")
+	(text "add zeners"
+		(exclude_from_sim no)
+		(at 110.744 20.066 0)
+		(effects
+			(font
+				(size 1.27 1.27)
+			)
+		)
+	)
 	(junction
 		(at 251.46 40.64)
