File: ControlBoard/ControlBoard/Control.kicad_sch (KiCad schematic)
At the start: 38 parts, among them IC1 TXB0104DR, IC2 ADS8688AIDBT, IC4 TXB0104DR, IC5 TXB0104DR, IC7 TXB0104DR, IC8 TXB0104DR, J1 Conn_01x02_Pin

Commit message: Hardware updates
Other:
- note added: "add filter caps here for all inputs"
- note added: "check extra pins"
Changed lines of the file:
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@@
 	(generator_version "9.0")
 	(paper "A4")
+	(text "check extra pins"
+		(exclude_from_sim no)
+		(at 68.834 50.292 0)
+		(effects
+			(font
+				(size 1.27 1.27)
+			)
+			(justify left)
+		)
+	)
 	(text "UART Debug Header"
 		(exclude_from_sim no)
@@
 		)
 	)
+	(text "add filter caps here for all inputs"
+		(exclude_from_sim no)
+		(at 69.596 191.77 0)
+		(effects
+			(font
+				(size 1.27 1.27)
+			)
+			(justify left)
+		)
+	)
