File: Boards/DynamicBrakeGrid/PowerStage.kicad_sch (KiCad schematic)
At the start: 38 parts, among them IC3 UCC27424QDRQ1, IC8 LM358DR, Q1 STWA75N60M6, Q2 STWA75N60M6, U6 ACS758xCB-200U-PFF

Commit message: Update DYBRK Schematic
Parts:
- removed C40: 100nF, Capacitor_SMD:C_1210_3225Metric_Pad1.33x2.70mm_HandSolder, symbol Device:C
- removed C47: 1nF, Capacitor_SMD:C_1210_3225Metric_Pad1.33x2.70mm_HandSolder, symbol Device:C
- removed FB3: FBMJ1608HS220NTR, InverterCom:BEADC1608X100N, symbol Device:FerriteBead
- removed H5, H6: 677-15ABPE, InverterCom:67715ABPE, symbol InverterCom:677-15ABPE
- removed Q1, Q2: STWA75N60M6, InverterCom:TO544P510X1580X2540-3P, symbol InverterCom:STWA75N60M6
- removed R54: 58, Resistor_SMD:R_1210_3225Metric_Pad1.30x2.65mm_HandSolder, symbol Device:R
- removed R55: 10k, Resistor_SMD:R_1210_3225Metric_Pad1.30x2.65mm_HandSolder, symbol Device:R
- removed R56: 1, Resistor_SMD:R_1210_3225Metric_Pad1.30x2.65mm_HandSolder, symbol Device:R
- removed R58: 0, Resistor_SMD:R_1210_3225Metric_Pad1.30x2.65mm_HandSolder, symbol Device:R
- added C16, C17, C18, C19: ALH82A750CB600, InverterCom:ALH82A750CB600, symbol InverterCom:ALH82A750CB600
- added Q1: ~, symbol InverterCom:FZ400R12KE4
- added Z10, Z11, Z9: 1SMB2EZ15_R1_00001, 1SMB2EZ15_R1_00001, symbol InverterCom:1SMB2EZ15_R1_00001
- R51: value 10k -> 1k
Connections:
- net Gate2 is gone; now on net Gate: IC3.5 (OUTB)
- net DC_LINK_V+: now also C16.1, C17.1, C18.1, C19.1
- net GND: now also Q1.5 (E), Z10.2 (A), Z11.2 (A), Z9.2 (A)
- net GNDPWR: now also C16.2, C17.2, C18.2, C19.2, Q1.2 (E)
- net at C38.2, C39.2: now also FB1.1, R53.2; no longer FB1.2, R53.1
- net CHOPPER_DRAIN: now reaches U6.5 (IP-)
- net CHOPPER_DRAIN: now also Q1.1 (C)
- net Gate1 renamed Gate
- net Gate: now also R53.1; no longer FB1.1
- new net: FB1.2, Q1.3 (G), Z10.1 (K), Z11.1 (K), Z9.1 (K)
Other:
- moved on the sheet: C38, C39, FB1, R51, R52, R53

Commit message: Update Dynamic Brake Board
Parts:
- added TP23, TP24, TP25, TP26, TP27, TP28: TestPoint, TestPoint:TestPoint_Loop_D2.54mm_Drill1.5mm_Beaded, symbol Connector:TestPoint
- Q1: footprint (none) -> InverterCom:FZ400R12KE4
- Z10, Z11, Z9: footprint 1SMB2EZ15_R1_00001 -> InverterCom:1SMB2EZ15_R1_00001
Connections:
- net Arduino_CurrentSense: now also TP27.1
- net GATE_PWM: now also TP28.1
- net GND: now also TP25.1
- net Gate: now also TP24.1
- net at C76.2, C79.1, IC8.3 (IN1+)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: now also TP26.1
- net at FB1.2, Q1.3 (G), Z10.1 (K)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: now also TP23.1

Commit message: Update Gate Resistor
Parts:
- R53: value 58 -> 10
Changed lines of the file:
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@@
 			)
 		)
-		(property "Value" "58"
+		(property "Value" "10"
 			(at 38.1 96.52 90)
 			(effects

Commit message: Generate Bill of Materials
Parts:
- Q1: value ~ -> FZ400R12KE4
- U6: value ACS758xCB-200U-PFF -> ACS758ECB-200U-PFF
Changed lines of the file:
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@@
 			)
 		)
-		(property "Value" "~"
+		(property "Value" "FZ400R12KE4"
 			(at 116.84 104.8992 0)
 			(effects
@@
 			)
 		)
-		(property "Value" "ACS758xCB-200U-PFF"
+		(property "Value" "ACS758ECB-200U-PFF"
 			(at 177.8 96.5514 0)
 			(effects

Commit message: Update Gate Driver to use non NDA BS Chip
Parts:
- added HS1: 567-125409, symbol Mechanical:Heatsink
Changed lines of the file:
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@@
+	)
+	(symbol
+		(lib_id "Mechanical:Heatsink")
+		(at 132.08 123.19 0)
+		(unit 1)
+		(exclude_from_sim yes)
+		(in_bom yes)
+		(on_board no)
+		(dnp no)
+		(fields_autoplaced yes)
+		(property "Reference" "HS1"
+			(at 135.89 120.0149 0)
+			(effects
+				(font
+					(size 1.27 1.27)
+				)
+				(justify left)
+			)
+		)
+		(property "Value" "567-125409"
+			(at 135.89 122.5549 0)
+			(effects
+				(font
+					(size 1.27 1.27)
+				)
+				(justify left)
+			)
+		)
+		(property "Footprint" ""
+			(at 132.3848 123.19 0)
+			(effects
+				(font
+					(size 1.27 1.27)
+				)
+				(hide yes)
+			)
+		)
+		(property "Datasheet" "~"
+			(at 132.3848 123.19 0)
+			(effects
+				(font
+					(size 1.27 1.27)
+				)
+				(hide yes)
+			)
+		)
+		(property "Description" "Heatsink"
+			(at 132.08 123.19 0)
+			(effects
+				(font
+					(size 1.27 1.27)
+				)
+				(hide yes)
+			)
+		)
+		(instances
+			(project ""
+				(path "/c99e0392-d1c3-4f46-a25d-449c454a3f3b/8cde10ba-b1fe-45d4-b2d9-70e5e14dd7c6"
+					(reference "HS1")
+					(unit 1)
+				)
+			)
+		)
 	)
 	(symbol

Commit message: Update Dybrk FW
Parts:
- added C100: 4.7uF, Capacitor_SMD:C_1210_3225Metric_Pad1.33x2.70mm_HandSolder, symbol Device:C
- added C99: 100pF, Capacitor_SMD:C_1210_3225Metric_Pad1.33x2.70mm_HandSolder, symbol Device:C
- C76: now fitted
Connections:
- net GND: now also C100.2, C99.2
- net at C76.2, C79.1, IC8.3 (IN1+)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: now also C100.1, C99.1
