File: Boards/IsolatedVoltageSensor/IsolatedVoltageAmplifier.kicad_sch (KiCad schematic)
At the start: 104 parts, among them IC1 TLV6001QDCKRQ1, IC11 TLV6001QDCKRQ1, IC12 TLV6001QDCKRQ1, IC2 TLV6001QDCKRQ1

Commit message: Finalize Voltage Sense Board
Parts:
- added FB1, FB2, FB3, FB4: FBMJ1608HS220NTR, InverterCom:BEADC1608X100N, symbol InverterCom:FBMJ1608HS220NTR
- added Z1, Z2, Z3, Z4: SZMMSZ4678T1G, InverterCom:SOD3716X135N, symbol InverterCom:SZMMSZ4678T1G
Connections:
- net +5V: no longer AT1.12 (VDD), AT2.12 (VDD), AT3.12 (VDD), AT4.12 (VDD), C35.1, C36.1, C41.2, C56.2, C57.1, C58.1, C68.2, C69.1, C70.1, C80.2, C81.1, C82.1
- net GNDPWR: now also Z1.2 (A), Z2.2 (A), Z3.2 (A), Z4.2 (A)
- net at AT1.6 (INP), C46.1, TP2.1: now also FB1.2, Z1.1 (K); no longer R37.1
- net at AT2.6 (INP), C49.1, TP7.1: now also FB2.2, Z2.1 (K); no longer R44.1
- net at AT3.6 (INP), C61.1, TP12.1: now also FB3.2, Z3.1 (K); no longer R50.1
- net at AT4.6 (INP), C73.1, TP17.1: now also FB4.2, Z4.1 (K); no longer R56.1
- new net: FB3.1, R50.1
- new net: FB4.1, R56.1
- new net: FB1.1, R37.1
- new net: FB2.1, R44.1
- new net +3.3V: AT1.12 (VDD), AT2.12 (VDD), AT3.12 (VDD), AT4.12 (VDD), C35.1, C36.1, C41.2, C56.2, C57.1, C58.1, C68.2, C69.1, C70.1, C80.2, C81.1, C82.1
Other:
- moved on the sheet: AT1, AT2, AT3, AT4, C35, C36, C38, C39, C40, C41, C42, C43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
