File: Boards/IsolatedVoltageSensor/PowerSupply.kicad_sch (KiCad schematic)
At the start: 0 parts

Commit message: Finalize Voltage Sense Board
Parts:
- added C1, C4: UVY1E102MPD1TD, InverterCom:CAPPRD500W60D1025H1750, symbol InverterCom:UVY1E102MPD1TD
- added PS1: R-78K3.3-1.0, InverterCom:R78K3310, symbol InverterCom:R-78K3.3-1.0
Connections:
- new net +3.3V: C4.1 (+), PS1.3 (+VOUT)
- new net +5V: C1.1 (+), PS1.1 (+VIN)
- new net GND: C1.2 (-), C4.2 (-), PS1.2 (GND)
