File: Boards/IsolatedVoltageSensor/Connectors.kicad_sch (KiCad schematic)
At the start: 6 parts, among them J1 Conn_01x10_Pin, J2 Conn_01x10_Pin

Commit message: Update
Connections:
- net +5V: now also J2.10 (Pin_10); no longer J2.1 (Pin_1)
- net DC_LINK_BUS_ISOLATED_VSENSE: now also J2.8 (Pin_8); no longer J2.3 (Pin_3)
- net DC_LINK_BUS_VSENSE: now also J1.9 (Pin_9); no longer J1.2 (Pin_2)
- net GND: now also J2.1 (Pin_1), J2.3 (Pin_3), J2.5 (Pin_5), J2.7 (Pin_7), J2.9 (Pin_9); no longer J2.10 (Pin_10), J2.2 (Pin_2), J2.4 (Pin_4), J2.6 (Pin_6), J2.8 (Pin_8)
- net GNDPWR: now also J1.2 (Pin_2), J1.4 (Pin_4), J1.6 (Pin_6), J1.8 (Pin_8); no longer J1.3 (Pin_3), J1.5 (Pin_5), J1.7 (Pin_7), J1.9 (Pin_9)
- net PHASE_U_ISOLATED_VSENSE: now also J2.2 (Pin_2); no longer J2.9 (Pin_9)
- net PHASE_U_VSENSE: now also J1.7 (Pin_7); no longer J1.4 (Pin_4)
- net PHASE_V_ISOLATED_VSENSE: now also J2.4 (Pin_4); no longer J2.7 (Pin_7)
- net PHASE_V_VSENSE: now also J1.5 (Pin_5); no longer J1.6 (Pin_6)
- net PHASE_W_ISOLATED_VSENSE: now also J2.6 (Pin_6); no longer J2.5 (Pin_5)
- net PHASE_W_VSENSE: now also J1.3 (Pin_3); no longer J1.8 (Pin_8)
