File: Boards/IsolatedVoltageSensor/IsolatedVoltageSensor.kicad_pcb (KiCad board)
At the start: 4 copper layers, 125 x 85 mm, 117 parts, among them IC1 TLV6001QDCKRQ1, IC11 TLV6001QDCKRQ1, IC12 TLV6001QDCKRQ1, IC2 TLV6001QDCKRQ1, J1 Conn_01x10_Pin, J2 Conn_01x10_Pin

Commit message: Finalize Voltage Sense Board
Parts:
- removed the G*** at (195.0, 131.0)
- added C1: UVY1E102MPD1TD, InverterCom:CAPPRD500W60D1025H1750, F.Cu at (191.0, 132.0)
- added C4: UVY1E102MPD1TD, InverterCom:CAPPRD500W60D1025H1750, F.Cu at (207.0, 125.5)
- added FB1: FBMJ1608HS220NTR, InverterCom:BEADC1608X100N, F.Cu at (117.5, 133.5)
- added FB2: FBMJ1608HS220NTR, InverterCom:BEADC1608X100N, F.Cu at (117.2, 115.0)
- added FB3: FBMJ1608HS220NTR, InverterCom:BEADC1608X100N, F.Cu at (118.5, 96.0)
- added FB4: FBMJ1608HS220NTR, InverterCom:BEADC1608X100N, F.Cu at (117.2, 76.5)
- added G***: LOGO, InverterCom:Char_AllelujahHaptism_20mm, F.Cu at (101.0, 118.0)
- added PS1: R-78K3.3-1.0, InverterCom:R78K3310, F.Cu at (192.0, 122.3)
- added Z1: SZMMSZ4678T1G, InverterCom:SOD3716X135N, F.Cu at (120.0, 137.5)
- added Z2: SZMMSZ4678T1G, InverterCom:SOD3716X135N, F.Cu at (120.0, 118.5)
- added Z3: SZMMSZ4678T1G, InverterCom:SOD3716X135N, F.Cu at (120.5, 99.5)
- added Z4: SZMMSZ4678T1G, InverterCom:SOD3716X135N, F.Cu at (120.0, 80.0)
- moved R37 9.00 mm to (111.5, 133.5)
- moved R44 8.55 mm to (112.0, 115.0)
- moved R56 8.00 mm to (112.0, 76.5)
- moved R50 7.00 mm to (113.5, 96.0)
- moved G*** 1.00 mm to (191.5, 80.0)
Connections:
- AT1 pad 12: +5V -> +3.3V
- AT2 pad 12: +5V -> +3.3V
- AT3 pad 12: +5V -> +3.3V
- AT4 pad 12: +5V -> +3.3V
- C35 pad 1: +5V -> +3.3V
- C36 pad 1: +5V -> +3.3V
- C41 pad 2: +5V -> +3.3V
- C56 pad 2: +5V -> +3.3V
- C57 pad 1: +5V -> +3.3V
- C58 pad 1: +5V -> +3.3V
- C68 pad 2: +5V -> +3.3V
- C69 pad 1: +5V -> +3.3V
- C70 pad 1: +5V -> +3.3V
- C80 pad 2: +5V -> +3.3V
- C81 pad 1: +5V -> +3.3V
- C82 pad 1: +5V -> +3.3V
- R37 pad 1: Net-(AT1-INP) -> Net-(FB1-Pad1)
- R44 pad 1: Net-(AT2-INP) -> Net-(FB2-Pad1)
- R50 pad 1: Net-(AT3-INP) -> Net-(FB3-Pad1)
- R56 pad 1: Net-(AT4-INP) -> Net-(FB4-Pad1)
Routing:
- net +3.3V: track 0.00 -> 179.5 mm, vias 0 -> 4
- net +5V: track 94.7 -> 42.8 mm, vias 8 -> 4
- net DC_LINK_BUS_VSENSE: track 67.5 -> 58.5 mm
- net PHASE_U_VSENSE: track 44.0 -> 35.5 mm
- net PHASE_V_VSENSE: track 33.0 -> 26.0 mm
- net Net-(AT1-INP): track 29.3 -> 35.2 mm
- net PHASE_W_VSENSE: track 57.1 -> 51.2 mm
- net Net-(AT2-INP): track 29.7 -> 35.2 mm
- net Net-(AT4-INP): track 29.7 -> 34.5 mm
- net Net-(AT3-INP): track 29.4 -> 33.8 mm
- net Net-(FB1-Pad1): track 0.00 -> 3.65 mm
- net Net-(FB4-Pad1): track 0.00 -> 2.85 mm
- net Net-(FB2-Pad1): track 0.00 -> 2.85 mm
- net Net-(FB3-Pad1): track 0.00 -> 2.15 mm
- net DC_LINK_BUS_ISOLATED_VSENSE: track 65.9 -> 64.4 mm
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- added copper zone on B.Cu, net GND
- added copper zone on In1.Cu, net GND
- added copper zone on B.Cu, net GNDPWR
- added copper zone on In1.Cu, net GNDPWR
- added copper zone on In2.Cu, net GNDPWR

Commit message: Update
Parts:
- moved TP9 17.5 mm to (200.0, 92.5)
- moved TP4 12.5 mm to (195.0, 107.5)
- moved TP14 8.00 mm to (196.0, 97.5)
- moved TP19 2.50 mm to (200.0, 102.5)
Connections:
- J1 pad 2: DC_LINK_BUS_VSENSE -> GNDPWR
- J1 pad 3: GNDPWR -> PHASE_W_VSENSE
- J1 pad 4: PHASE_U_VSENSE -> GNDPWR
- J1 pad 5: GNDPWR -> PHASE_V_VSENSE
- J1 pad 6: PHASE_V_VSENSE -> GNDPWR
- J1 pad 7: GNDPWR -> PHASE_U_VSENSE
- J1 pad 8: PHASE_W_VSENSE -> GNDPWR
- J1 pad 9: GNDPWR -> DC_LINK_BUS_VSENSE
- J2 pad 1: +5V -> GND
- J2 pad 10: GND -> +5V
- J2 pad 2: GND -> PHASE_U_ISOLATED_VSENSE
- J2 pad 3: DC_LINK_BUS_ISOLATED_VSENSE -> GND
- J2 pad 4: GND -> PHASE_V_ISOLATED_VSENSE
- J2 pad 5: PHASE_W_ISOLATED_VSENSE -> GND
- J2 pad 6: GND -> PHASE_W_ISOLATED_VSENSE
- J2 pad 7: PHASE_V_ISOLATED_VSENSE -> GND
- J2 pad 8: GND -> DC_LINK_BUS_ISOLATED_VSENSE
- J2 pad 9: PHASE_U_ISOLATED_VSENSE -> GND
Routing:
- net DC_LINK_BUS_VSENSE: track 58.5 -> 41.1 mm
- net PHASE_U_ISOLATED_VSENSE: track 30.4 -> 47.7 mm
- net PHASE_W_VSENSE: track 51.2 -> 37.1 mm
- net DC_LINK_BUS_ISOLATED_VSENSE: track 64.4 -> 52.0 mm
- net PHASE_U_VSENSE: track 35.5 -> 28.0 mm
- net PHASE_V_ISOLATED_VSENSE: track 36.6 -> 29.4 mm, vias 2 -> 0
- net PHASE_V_VSENSE: track 26.0 -> 23.5 mm
- net PHASE_W_ISOLATED_VSENSE: track 56.1 -> 58.3 mm
- net GND: track 6.31 -> 7.47 mm
- net GNDPWR: vias 304 -> 296
