File: Boards/GateDriver/Connectors.kicad_sch (KiCad schematic)
At the start: 10 parts, among them J1 1548129, J3 1548129, J4 5-106505-2, J5 1987724, J6 1987724, J7 1987724

Commit message: Update Gate Driver to use non NDA BS Chip
Parts:
- J4: footprint 5-106505-2_3 -> InverterCom:5-106505-2_3
Changed lines of the file:
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@@
 			)
 		)
-		(property "Footprint" "5-106505-2_3"
+		(property "Footprint" "InverterCom:5-106505-2_3"
 			(at 52.07 117.78 0)
 			(effects
