File: Boards/HMI/Control.kicad_sch (KiCad schematic)
At the start: 24 parts, among them IC1 ISO1042BDWVR, IC6 MCP2515-e_ST, Y1 8MHz

Commit message: Update Gate Driver to use non NDA BS Chip
Parts:
- Y1: footprint Crystal:Crystal_SMD_7050-2Pin_7.0x5.0mm_HandSoldering -> Crystal:Crystal_HC49-4H_Vertical
Changed lines of the file:
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@@
 			)
 		)
-		(property "Footprint" "Crystal:Crystal_SMD_7050-2Pin_7.0x5.0mm_HandSoldering"
+		(property "Footprint" "Crystal:Crystal_HC49-4H_Vertical"
 			(at 167.64 77.47 0)
 			(effects
