File: Boards/PowerBoard/PowerAssembly.kicad_sch (KiCad schematic)
At the start: 54 parts

Commit message: Update Layouts
Other:
- note removed: "add zeners"
Changed lines of the file:
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@@
 	(generator_version "9.0")
 	(paper "A4")
-	(text "add zeners"
-		(exclude_from_sim no)
-		(at 110.744 20.066 0)
-		(effects
-			(font
-				(size 1.27 1.27)
-			)
-		)
-	)
 	(junction
 		(at 251.46 40.64)
