File: Boards/PowerBoard/PowerBoard.kicad_pcb (KiCad board)
At the start: 4 copper layers, 430 x 310 mm, 164 parts, among them IC10 ACS772ECB-400B-PFF-T, IC3 ACS772ECB-400B-PFF-T, IC4 ACS772ECB-400B-PFF-T, IC5 ACS772ECB-400B-PFF-T, IC6 ACS772ECB-400B-PFF-T, IC7 ACS772ECB-400B-PFF-T, IC8 ACS772ECB-400B-PFF-T, IC9 ACS772ECB-400B-PFF-T, J6 L717SDB25PA4CH3R, J8 Conn_01x10_Socket, J9 Conn_01x10_Socket

Commit message: Add Zeners to Power Board
Parts:
- added C35: 1nF, Capacitor_SMD:C_1210_3225Metric_Pad1.33x2.70mm_HandSolder, B.Cu at (-80.5, 118.5)
- added C36: 10nF, Capacitor_SMD:C_1210_3225Metric_Pad1.33x2.70mm_HandSolder, B.Cu at (-85.0, 118.5)
- added C38: 100nF, Capacitor_SMD:C_1210_3225Metric_Pad1.33x2.70mm_HandSolder, B.Cu at (-89.5, 118.5)
- added C39: 1nF, Capacitor_SMD:C_1210_3225Metric_Pad1.33x2.70mm_HandSolder, B.Cu at (-88.2, 129.6)
- added C40: 10nF, Capacitor_SMD:C_1210_3225Metric_Pad1.33x2.70mm_HandSolder, B.Cu at (-83.7, 129.6)
- added C41: 100nF, Capacitor_SMD:C_1210_3225Metric_Pad1.33x2.70mm_HandSolder, B.Cu at (-79.5, 129.6)
- added C42: 1nF, Capacitor_SMD:C_1210_3225Metric_Pad1.33x2.70mm_HandSolder, B.Cu at (-65.5, 132.0)
- added C43: 10nF, Capacitor_SMD:C_1210_3225Metric_Pad1.33x2.70mm_HandSolder, B.Cu at (-69.9, 132.0)
- added C44: 100nF, Capacitor_SMD:C_1210_3225Metric_Pad1.33x2.70mm_HandSolder, B.Cu at (-74.2, 132.0)
- added C45: 1nF, Capacitor_SMD:C_1210_3225Metric_Pad1.33x2.70mm_HandSolder, B.Cu at (-83.7, 138.4)
- added C46: 10nF, Capacitor_SMD:C_1210_3225Metric_Pad1.33x2.70mm_HandSolder, B.Cu at (-79.3, 138.4)
- added C47: 100nF, Capacitor_SMD:C_1210_3225Metric_Pad1.33x2.70mm_HandSolder, B.Cu at (-75.1, 138.4)
- added C48: 1nF, Capacitor_SMD:C_1210_3225Metric_Pad1.33x2.70mm_HandSolder, B.Cu at (-62.5, 200.5)
- added C49: 10nF, Capacitor_SMD:C_1210_3225Metric_Pad1.33x2.70mm_HandSolder, B.Cu at (-53.9, 200.5)
- added C50: 100nF, Capacitor_SMD:C_1210_3225Metric_Pad1.33x2.70mm_HandSolder, B.Cu at (-58.1, 200.5)
- added C51: 1nF, Capacitor_SMD:C_1210_3225Metric_Pad1.33x2.70mm_HandSolder, B.Cu at (-62.5, 190.5)
- added C52: 10nF, Capacitor_SMD:C_1210_3225Metric_Pad1.33x2.70mm_HandSolder, B.Cu at (-58.0, 190.5)
- added C53: 100nF, Capacitor_SMD:C_1210_3225Metric_Pad1.33x2.70mm_HandSolder, B.Cu at (-53.5, 190.6)
- added C54: 1nF, Capacitor_SMD:C_1210_3225Metric_Pad1.33x2.70mm_HandSolder, B.Cu at (-62.5, 181.5)
- added C55: 10nF, Capacitor_SMD:C_1210_3225Metric_Pad1.33x2.70mm_HandSolder, B.Cu at (-53.8, 181.5)
- added C56: 100nF, Capacitor_SMD:C_1210_3225Metric_Pad1.33x2.70mm_HandSolder, B.Cu at (-58.0, 181.5)
- added C57: 1nF, Capacitor_SMD:C_1210_3225Metric_Pad1.33x2.70mm_HandSolder, B.Cu at (-62.4, 170.5)
- added C58: 10nF, Capacitor_SMD:C_1210_3225Metric_Pad1.33x2.70mm_HandSolder, B.Cu at (-53.8, 170.5)
- added C59: 100nF, Capacitor_SMD:C_1210_3225Metric_Pad1.33x2.70mm_HandSolder, B.Cu at (-58.0, 170.5)
- added C60: 1nF, Capacitor_SMD:C_1210_3225Metric_Pad1.33x2.70mm_HandSolder, B.Cu at (-76.0, 124.0)
- added C61: 10nF, Capacitor_SMD:C_1210_3225Metric_Pad1.33x2.70mm_HandSolder, B.Cu at (-71.8, 124.0)
- added C62: 100nF, Capacitor_SMD:C_1210_3225Metric_Pad1.33x2.70mm_HandSolder, B.Cu at (-67.5, 124.0)
- added C63: 1nF, Capacitor_SMD:C_1210_3225Metric_Pad1.33x2.70mm_HandSolder, B.Cu at (-80.2, 144.0)
- added C64: 10nF, Capacitor_SMD:C_1210_3225Metric_Pad1.33x2.70mm_HandSolder, B.Cu at (-88.8, 144.0)
- added C65: 100nF, Capacitor_SMD:C_1210_3225Metric_Pad1.33x2.70mm_HandSolder, B.Cu at (-84.5, 144.0)
- added C66: 1nF, Capacitor_SMD:C_1210_3225Metric_Pad1.33x2.70mm_HandSolder, B.Cu at (-72.1, 146.1)
- added C67: 10nF, Capacitor_SMD:C_1210_3225Metric_Pad1.33x2.70mm_HandSolder, B.Cu at (-76.3, 146.1)
- added C68: 100nF, Capacitor_SMD:C_1210_3225Metric_Pad1.33x2.70mm_HandSolder, B.Cu at (-68.0, 146.0)
- added C69: 1nF, Capacitor_SMD:C_1210_3225Metric_Pad1.33x2.70mm_HandSolder, B.Cu at (-80.5, 150.9)
- added C70: 10nF, Capacitor_SMD:C_1210_3225Metric_Pad1.33x2.70mm_HandSolder, B.Cu at (-84.8, 150.9)
- added C71: 100nF, Capacitor_SMD:C_1210_3225Metric_Pad1.33x2.70mm_HandSolder, B.Cu at (-89.0, 150.9)
- added Z1: 1SMB5956BT3G, InverterCom:DIOM5436X247N, B.Cu at (57.5, 226.0)
- added Z10: 1SMB5956BT3G, InverterCom:DIOM5436X247N, B.Cu at (287.0, 211.5)
- added Z11: 1SMB5956BT3G, InverterCom:DIOM5436X247N, B.Cu at (287.0, 219.0)
- added Z12: 1SMB5956BT3G, InverterCom:DIOM5436X247N, B.Cu at (287.0, 226.5)
- added Z13: 1SMB5956BT3G, InverterCom:DIOM5436X247N, B.Cu at (57.5, 35.3)
- added Z14: 1SMB5956BT3G, InverterCom:DIOM5436X247N, B.Cu at (57.5, 43.0)
- added Z15: 1SMB5956BT3G, InverterCom:DIOM5436X247N, B.Cu at (57.5, 50.5)
- added Z16: 1SMB5956BT3G, InverterCom:DIOM5436X247N, B.Cu at (57.5, 58.0)
- added Z17: 1SMB5956BT3G, InverterCom:DIOM5436X247N, B.Cu at (287.0, 35.3)
- added Z18: 1SMB5956BT3G, InverterCom:DIOM5436X247N, B.Cu at (287.0, 43.0)
- added Z19: 1SMB5956BT3G, InverterCom:DIOM5436X247N, B.Cu at (287.0, 50.5)
- added Z2: 1SMB5956BT3G, InverterCom:DIOM5436X247N, B.Cu at (57.5, 218.5)
- added Z20: 1SMB5956BT3G, InverterCom:DIOM5436X247N, B.Cu at (287.0, 58.0)
- added Z21: 1SMB5956BT3G, InverterCom:DIOM5436X247N, B.Cu at (172.0, 35.0)
- added Z22: 1SMB5956BT3G, InverterCom:DIOM5436X247N, B.Cu at (172.0, 42.5)
- added Z23: 1SMB5956BT3G, InverterCom:DIOM5436X247N, B.Cu at (172.0, 50.0)
- added Z24: 1SMB5956BT3G, InverterCom:DIOM5436X247N, B.Cu at (172.0, 57.5)
- added Z3: 1SMB5956BT3G, InverterCom:DIOM5436X247N, B.Cu at (57.5, 211.0)
- added Z4: 1SMB5956BT3G, InverterCom:DIOM5436X247N, B.Cu at (57.5, 203.5)
- added Z5: 1SMB5956BT3G, InverterCom:DIOM5436X247N, B.Cu at (172.0, 204.0)
- added Z6: 1SMB5956BT3G, InverterCom:DIOM5436X247N, B.Cu at (172.0, 211.5)
- added Z7: 1SMB5956BT3G, InverterCom:DIOM5436X247N, B.Cu at (172.0, 219.0)
- added Z8: 1SMB5956BT3G, InverterCom:DIOM5436X247N, B.Cu at (172.0, 226.5)
- added Z9: 1SMB5956BT3G, InverterCom:DIOM5436X247N, B.Cu at (287.0, 204.0)
- C19, C21, C22, C23, C24, C25, C26, C27, C28, C29, C30, C31, C32, C33, C34, C37, R1, R2, R3, R4, R5, R6, R7, R8: moved to B.Cu
- moved G*** 179.7 mm to (-2.50, 142.0)
- moved C28 39.3 mm to (283.5, 124.0), turned to 0 degrees
- moved C23 38.1 mm to (-67.5, 36.0), turned to -90 degrees
- moved C29 36.8 mm to (53.0, 123.5), turned to 0 degrees
- moved C30 34.5 mm to (167.9, 124.0), turned to 0 degrees
- moved C33 32.1 mm to (168.0, 116.5), turned to 0 degrees
- moved IC4 30.6 mm to (-64.3, 35.6), turned to -90 degrees
- moved R1 28.8 mm to (-58.5, 41.0)
- moved R8 27.8 mm to (289.0, 117.5)
- moved C27 27.4 mm to (283.5, 117.0), turned to 0 degrees
- moved R6 27.2 mm to (174.0, 117.5)
- moved C34 26.9 mm to (-60.0, 36.0)
- moved IC6 26.6 mm to (52.6, 120.8), turned to 0 degrees
- moved IC8 26.6 mm to (167.6, 120.8), turned to 0 degrees
- moved IC10 26.5 mm to (283.1, 120.8), turned to 0 degrees
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Connections:
- IC10 pad 4: PHASE_W -> PHASE_W_OUT
- IC10 pad 5: PHASE_W_OUT -> PHASE_W
- IC4 pad 4: DC_LINK_BUS -> DC_LINK_BUS_IN
- IC4 pad 5: DC_LINK_BUS_IN -> DC_LINK_BUS
- IC6 pad 4: PHASE_U -> PHASE_U_OUT
- IC6 pad 5: PHASE_U_OUT -> PHASE_U
- IC8 pad 4: PHASE_V -> PHASE_V_OUT
- IC8 pad 5: PHASE_V_OUT -> PHASE_V
Routing:
- net +5V: track 895.0 -> 1060.2 mm, vias 9 -> 5
- net GND: track 735.2 -> 883.6 mm, vias 11 -> 6
- net GNDPWR: track 92.8 -> 199.2 mm
- net DC_LINK_BUS: track 182.1 -> 220.7 mm
- net PHASE_V: track 163.7 -> 189.3 mm
- net PHASE_W: track 266.8 -> 292.4 mm
- net PHASE_U: track 41.2 -> 65.8 mm
- net PHASE_U_ISENSE: track 265.5 -> 244.8 mm, vias 3 -> 2
- net PHASE_V_ISENSE: track 377.2 -> 360.1 mm, vias 3 -> 2
- net PHASE_W_ISENSE: track 490.3 -> 478.1 mm
- net PHASE_W_VSENSE: track 19.0 -> 31.0 mm, vias 0 -> 1
- net PHASE_V_VSENSE: track 33.0 -> 44.6 mm
- net PHASE_U_VSENSE: track 48.4 -> 59.7 mm
- net DC_LINK_BUS_VSENSE: track 63.1 -> 74.3 mm
- net Net-(IC3-VIOUT): track 15.1 -> 4.93 mm
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
Commit message: Update Layouts
Changed lines of the file:
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@@
 	(gr_poly
 		(pts
-			(xy -81.5 17.5) (xy -76.5 13) (xy 277 13) (xy 277 30) (xy -52 30) (xy -52 30) (xy -81.5 30)
+			(xy -81.5 17.5) (xy -76.5 13) (xy 277 13) (xy 277 30) (xy -52 30) (xy -81.5 30)
 		)
 		(stroke
@@
 		(layer "F.Mask")
 	)
+	(gr_rect
+		(start -82 45)
+		(end -73 60)
+		(stroke
+			(width 0.1)
+			(type solid)
+		)
+		(fill yes)
+		(layer "F.Mask")
+	)
+	(gr_rect
+		(start -48.5 45)
+		(end -39.5 60)
+		(stroke
+			(width 0.1)
+			(type solid)
+		)
+		(fill yes)
+		(layer "F.Mask")
+	)
 	(gr_poly
 		(pts
@@
 		(polygon
 			(pts
-				(xy -85 47.5) (xy -82.5 45) (xy -72.5 45) (xy -67.5 55) (xy -55 55) (xy -50 45) (xy -40 45) (xy -37.5 47.5)
+				(xy -85 47.5) (xy -82.5 45) (xy -72.5 45) (xy -67.5 55) (xy -55 55) (xy -50 45) (xy -39 45) (xy -37.5 46.5)
 				(xy -37.5 60) (xy -37.5 62.5) (xy -87.5 62.5) (xy -87.5 60) (xy -85 57.5)
 			)

Commit message: Update
Routing:
- net PHASE_W_VSENSE: vias 1 -> 2
- net GNDPWR: vias 4 -> 187
